Commit message: Added robotiq gripper

File: grizzly_ur10_description/urdf/gripper.urdf.xacro (robot description, xacro)
@@ -26,6 +26,23 @@
 -->
 <robot xmlns:xacro="http://ros.org/wiki/xacro" name="grizzly_ur10">
-  <xacro:include filename="$(find grizzly_description)/urdf/base.urdf.xacro" />
-  <xacro:include filename="$(find grizzly_ur10_description)/urdf/manipulator.urdf.xacro" />
-  <xacro:include filename="$(find grizzly_ur10_description/urdf/gripper.urdf.xacro" />
+  <xacro:property name="reflect" value="-1" />
+ <xacro:include filename="$(find ur_description)/urdf/gazebo.urdf.xacro" />
+  <xacro:include filename="$(find ur_description)/urdf/ur10.urdf.xacro" />
+  <xacro:include filename="$(find robotiq_s_model_visualization)/cfg/s-model_articulated_macro.urdf.xacro" />
+  <!-- Spawn arm -->
+  <xacro:ur10_robot prefix="ur10_arm_" joint_limited="true"/>
+  <!-- <xacro:ur10_robot prefix="" joint_limited="true" /> -->
+  <joint name="grizzly_ur10_joint" type="fixed">
+    <parent link="sensor_anchor_link" />
+    <child link="ur10_arm_base_link" />
+    <origin xyz="0.65 ${reflect*0.21} 0.03" rpy="0.0 0.0 ${-pi/2}" />
+  </joint>
+  <!-- Spawn gripper -->
+  <xacro:s-model_articulated prefix="robotiq_"/>
+  <!-- Add robotiq gripper -->
+  <joint name="ee_joint" type="fixed">
+      <parent link="ee_link"/>
+      <child link="robotiq_palm"/>
+      <origin xyz="0 0 0" rpy="0 0 0" />
+  </joint>
 </robot>
