Commit message: Moved center of arm

File: grizzly_ur10_description/urdf/ur10_arm.urdf.xacro (robot description, xacro)
@@ -36,5 +36,5 @@
     <parent link="sensor_anchor_link" />
     <child link="ur10_arm_base_link" />
-    <origin xyz="0.65 ${reflect*0.21} 0.03" rpy="0.0 0.0 ${-pi/2}" />
+    <origin xyz="0.65 ${reflect*0.01} 0.03" rpy="0.0 0.0 ${-pi/2}" />
   </joint>
   <!-- Gazebo references for self collide -->

File: grizzly_ur10_gazebo/objects/cube_yellow.urdf (robot description, URDF)
Before this commit: robot simple_box, 1 links, 0 joints
Links:
- link my_box: geometry collision box size=0.04 0.04 0.04; visual box size=0.09 0.09 0.09
