Commit message: Added kinect model to sim

File: grizzly_ur10_description/urdf/grizzly_ur10_kinect.gazebo.xacro (robot description, xacro)
@@ -18,4 +18,31 @@
     <origin xyz="0 0 0" rpy="0 0 0"/>
 </joint>
+<!-- Adding the actual kinect model -->
+<link name="grizzly_ur10_kinect_link">
+	<visual>
+		<origin xyz="0 0 0" rpy="0 0 ${M_PI/2}"/>
+		<geometry>
+		<mesh filename="package://grizzly_ur10_description/meshes/sensors/kinect.dae"/>
+		</geometry>
+	</visual>
+	<collision>
+		<origin xyz="0.0 0.0 0.0" rpy="0 0 0"/>
+		<geometry>
+		<box size="0.07271 0.27794 0.073"/>
+		</geometry>
+	</collision>
+	<inertial>
+		<mass value="0.001" />
+		<origin xyz="0 0 0" />
+		<inertia ixx="0.0001" ixy="0.0" ixz="0.0"
+		iyy="0.0001" iyz="0.0"
+		izz="0.0001" />
+	</inertial>
+</link>
+<joint name="grizzly_ur10_kinect_joint" type="fixed">
+    <parent link="grizzly_ur10_kinect_frame"/>
+    <child link="grizzly_ur10_kinect_link"/>
+    <origin xyz="0 0 0" rpy="0 0 0"/>
+</joint>
 <!-- Add the kinect to the grizzly_ur10 project. This macro looks for ${name}_frame as its target frame. -->
 <xacro:kinect_camera_gazebo_v0 name="grizzly_ur10_kinect"/>

Commit message: Added the thingz

File: grizzly_ur10_description/urdf/grizzly_ur10_kinect.gazebo.xacro (robot description, xacro)
@@ -40,8 +40,9 @@
 	</inertial>
 </link>
+<!-- Connect kinect to robot -->
 <joint name="grizzly_ur10_kinect_joint" type="fixed">
     <parent link="grizzly_ur10_kinect_frame"/>
     <child link="grizzly_ur10_kinect_link"/>
-    <origin xyz="0 0 0" rpy="0 0 0"/>
+    <origin xyz="0.9 0 0" rpy="0 0 0"/>
 </joint>
 <!-- Add the kinect to the grizzly_ur10 project. This macro looks for ${name}_frame as its target frame. -->

Commit message: positioning like its a css website

File: grizzly_ur10_description/urdf/grizzly_ur10_kinect.gazebo.xacro (robot description, xacro)
@@ -10,5 +10,5 @@
     <parent link="sensor_anchor_link"/>
     <child link="grizzly_ur10_kinect_frame"/>
-    <origin xyz="0 0 0" rpy="0 0 0"/>
+    <origin xyz="0.9 0 0" rpy="0 0 0"/>
 </joint>
 <!-- Optical frame addition -->
@@ -44,5 +44,5 @@
     <parent link="grizzly_ur10_kinect_frame"/>
     <child link="grizzly_ur10_kinect_link"/>
-    <origin xyz="0.9 0 0" rpy="0 0 0"/>
+    <origin xyz="0 0 0" rpy="0 0 0"/>
 </joint>
 <!-- Add the kinect to the grizzly_ur10 project. This macro looks for ${name}_frame as its target frame. -->

Commit message: Modified frame translation

File: grizzly_ur10_description/urdf/grizzly_ur10_kinect.gazebo.xacro (robot description, xacro)
@@ -10,5 +10,5 @@
     <parent link="sensor_anchor_link"/>
     <child link="grizzly_ur10_kinect_frame"/>
-    <origin xyz="0.9 0 0" rpy="0 0 0"/>
+    <origin xyz="0.9 0 0" rpy="0 0 ${M_PI/2}"/>
 </joint>
 <!-- Optical frame addition -->
@@ -16,5 +16,5 @@
     <parent link="sensor_anchor_link"/>
     <child link="grizzly_ur10_kinect_optical_frame"/>
-    <origin xyz="0 0 0" rpy="0 0 0"/>
+    <origin xyz="0.9 0 0" rpy="0 0 ${M_PI/2}"/>
 </joint>
 <!-- Adding the actual kinect model -->

Commit message: Updated

File: grizzly_ur10_description/urdf/grizzly_ur10_kinect.gazebo.xacro (robot description, xacro)
@@ -8,13 +8,13 @@
 <!-- Kinect frame addition -->
 <joint name="grizzly_ur10_kinect_frame_joint" type="fixed">
-    <parent link="sensor_anchor_link"/>
+    <parent link="grizzly_ur10_kinect_link"/>
     <child link="grizzly_ur10_kinect_frame"/>
-    <origin xyz="0.9 0 0" rpy="0 0 ${M_PI/2}"/>
+    <origin xyz="0.9 0 0" rpy="0 0 0"/>
 </joint>
 <!-- Optical frame addition -->
 <joint name="grizzly_ur10_kinect_optical_frame_joint" type="fixed">
-    <parent link="sensor_anchor_link"/>
+    <parent link="grizzly_ur10_kinect_link"/>
     <child link="grizzly_ur10_kinect_optical_frame"/>
-    <origin xyz="0.9 0 0" rpy="0 0 ${M_PI/2}"/>
+    <origin xyz="0.9 0 0" rpy="0 0 0"/>
 </joint>
 <!-- Adding the actual kinect model -->
@@ -42,5 +42,5 @@
 <!-- Connect kinect to robot -->
 <joint name="grizzly_ur10_kinect_joint" type="fixed">
-    <parent link="grizzly_ur10_kinect_frame"/>
+    <parent link="sensor_anchor_link"/>
     <child link="grizzly_ur10_kinect_link"/>
     <origin xyz="0 0 0" rpy="0 0 0"/>

Commit message: updated

File: grizzly_ur10_description/urdf/grizzly_ur10_kinect.gazebo.xacro (robot description, xacro)
@@ -10,5 +10,5 @@
     <parent link="grizzly_ur10_kinect_link"/>
     <child link="grizzly_ur10_kinect_frame"/>
-    <origin xyz="0.9 0 0" rpy="0 0 0"/>
+    <origin xyz="0 0 0" rpy="0 0 0"/>
 </joint>
 <!-- Optical frame addition -->
@@ -16,5 +16,5 @@
     <parent link="grizzly_ur10_kinect_link"/>
     <child link="grizzly_ur10_kinect_optical_frame"/>
-    <origin xyz="0.9 0 0" rpy="0 0 0"/>
+    <origin xyz="0 0 0" rpy="0 0 0"/>
 </joint>
 <!-- Adding the actual kinect model -->
@@ -44,5 +44,5 @@
     <parent link="sensor_anchor_link"/>
     <child link="grizzly_ur10_kinect_link"/>
-    <origin xyz="0 0 0" rpy="0 0 0"/>
+    <origin xyz="0.9 0 0" rpy="0 0 0"/>
 </joint>
 <!-- Add the kinect to the grizzly_ur10 project. This macro looks for ${name}_frame as its target frame. -->

Commit message: closer

File: grizzly_ur10_description/urdf/grizzly_ur10_kinect.gazebo.xacro (robot description, xacro)
@@ -10,5 +10,5 @@
     <parent link="grizzly_ur10_kinect_link"/>
     <child link="grizzly_ur10_kinect_frame"/>
-    <origin xyz="0 0 0" rpy="0 0 0"/>
+    <origin xyz="0 0 0" rpy="-1.57 0 -1.57"/>
 </joint>
 <!-- Optical frame addition -->
@@ -16,5 +16,5 @@
     <parent link="grizzly_ur10_kinect_link"/>
     <child link="grizzly_ur10_kinect_optical_frame"/>
-    <origin xyz="0 0 0" rpy="0 0 0"/>
+    <origin xyz="0 0 0" rpy="-1.57 0 -1.57"/>
 </joint>
 <!-- Adding the actual kinect model -->

Commit message: I HATE TF AND RVIZ

File: grizzly_ur10_description/urdf/grizzly_ur10_kinect.gazebo.xacro (robot description, xacro)
@@ -7,19 +7,20 @@
 <link name="grizzly_ur10_kinect_optical_frame"/>
 <!-- Kinect frame addition -->
-<joint name="grizzly_ur10_kinect_frame_joint" type="fixed">
+<!-- <joint name="grizzly_ur10_kinect_frame_joint" type="fixed">
     <parent link="grizzly_ur10_kinect_link"/>
     <child link="grizzly_ur10_kinect_frame"/>
-    <origin xyz="0 0 0" rpy="-1.57 0 -1.57"/>
+    <origin xyz="0 0 0" rpy="0 0 ${M_PI/2}"/>
 </joint>
+ -->
 <!-- Optical frame addition -->
-<joint name="grizzly_ur10_kinect_optical_frame_joint" type="fixed">
+<!-- <joint name="grizzly_ur10_kinect_optical_frame_joint" type="fixed">
     <parent link="grizzly_ur10_kinect_link"/>
     <child link="grizzly_ur10_kinect_optical_frame"/>
-    <origin xyz="0 0 0" rpy="-1.57 0 -1.57"/>
-</joint>
+    <origin xyz="0 0 0" rpy="0 0 0"/>
+</joint> -->
 <!-- Adding the actual kinect model -->
 <link name="grizzly_ur10_kinect_link">
 	<visual>
-		<origin xyz="0 0 0" rpy="0 0 ${M_PI/2}"/>
+		<origin xyz="0 0 0" rpy="-${M_PI/2} 0 ${M_PI}"/>
 		<geometry>
 		<mesh filename="package://grizzly_ur10_description/meshes/sensors/kinect.dae"/>

Commit message: Sensor  now shows in a straight line

File: grizzly_ur10_description/urdf/grizzly_ur10_kinect.gazebo.xacro (robot description, xacro)
@@ -7,16 +7,15 @@
 <link name="grizzly_ur10_kinect_optical_frame"/>
 <!-- Kinect frame addition -->
-<!-- <joint name="grizzly_ur10_kinect_frame_joint" type="fixed">
+<joint name="grizzly_ur10_kinect_frame_joint" type="fixed">
     <parent link="grizzly_ur10_kinect_link"/>
     <child link="grizzly_ur10_kinect_frame"/>
-    <origin xyz="0 0 0" rpy="0 0 ${M_PI/2}"/>
+    <origin xyz="0 0 0" rpy="0 0 0"/>
 </joint>
- -->
 <!-- Optical frame addition -->
-<!-- <joint name="grizzly_ur10_kinect_optical_frame_joint" type="fixed">
-    <parent link="grizzly_ur10_kinect_link"/>
+<joint name="grizzly_ur10_kinect_optical_frame_joint" type="fixed">
+    <parent link="grizzly_ur10_kinect_frame"/>
     <child link="grizzly_ur10_kinect_optical_frame"/>
-    <origin xyz="0 0 0" rpy="0 0 0"/>
-</joint> -->
+    <origin xyz="0 0 0" rpy="0 0 -${M_PI/2}"/>
+</joint>
 <!-- Adding the actual kinect model -->
 <link name="grizzly_ur10_kinect_link">
@@ -45,5 +44,5 @@
     <parent link="sensor_anchor_link"/>
     <child link="grizzly_ur10_kinect_link"/>
-    <origin xyz="0.9 0 0" rpy="0 0 0"/>
+    <origin xyz="0.9 0 0" rpy="${M_PI/2} ${M_PI} ${M_PI/2}"/>
 </joint>
 <!-- Add the kinect to the grizzly_ur10 project. This macro looks for ${name}_frame as its target frame. -->
