Commit message: Working version of grizzly_ur10

File: grizzly_ur10_description/urdf/grizzly_ur10_hokuyo.gazebo.xacro (robot description, xacro)
@@ -5,6 +5,6 @@
 <xacro:include filename="$(find pr2_description)/urdf/common.xacro"/>
 <!-- Add laser -->
-<xacro:hokuyo_lx30_laser_v0 name="grizzly_ur10_hokyuo" parent="sensor_anchor" ros_topic="scan" update_rate="100" min_angle="0" max_angle="180">
-    <origin xyz="0.9 0 0" rpy="0 0 0"/>
+<xacro:hokuyo_lx30_laser_v0 name="grizzly_ur10_hokuyo" parent="sensor_anchor" ros_topic="scan" update_rate="100" min_angle="0" max_angle="180">
+    <origin xyz="1.0 0 -0.1" rpy="0 0 0"/>
 </xacro:hokuyo_lx30_laser_v0>
 </robot>

File: grizzly_ur10_description/urdf/grizzly_ur10_kinect.gazebo.xacro (robot description, xacro)
@@ -6,5 +6,5 @@
 <!-- Add kinect -->
 <xacro:kinect_camera_v0 name="grizzly_ur10_kinect" parent="sensor_anchor_link">
-    <origin xyz="0.9 0 0" rpy="0 0 0"/>
+    <origin xyz="0.5 0 0.4" rpy="0 ${M_PI/9} 0"/>
 </xacro:kinect_camera_v0>
 <gazebo reference="grizzly_ur10_kinect_link">
