Commit message: Removed double macro of robotiq grpiper bug

File: grizzly_ur10_description/urdf/robotiq_hand.urdf.xacro (robot description, xacro)
@@ -725,6 +725,3 @@
     <!-- end of joint list -->
   </xacro:macro>
- <xacro:robotiq_hand prefix="" reflect="1" parent="ur10_arm_ee_link">
-      <origin xyz="0 0 0" rpy="0 0 0"/>
-   </xacro:robotiq_hand>
 </robot>

Commit message: Updated robotiq urdf

File: grizzly_ur10_description/urdf/robotiq_hand.urdf.xacro (robot description, xacro)
@@ -648,5 +648,5 @@
         <visual>
           <geometry>
-            <mesh filename="package://robotiq-s-model_visualization/meshes/s-model_articulated/visual/palm.STL" />
+            <mesh filename="package://robotiq_s_model_visualization/meshes/s-model_articulated/visual/palm.STL" />
           </geometry>
           <material name="green">
