Commit message: Renaming to make more sense

File: grizzly_ur10_description/urdf/robotiq_gripper.urdf.xacro (robot description, xacro)
@@ -26,6 +26,15 @@
 -->
 <robot xmlns:xacro="http://ros.org/wiki/xacro" name="grizzly_ur10">
-  <xacro:include filename="$(find grizzly_description)/urdf/base.urdf.xacro" />
-  <xacro:include filename="$(find grizzly_ur10_description)/urdf/ur10_arm.urdf.xacro" />
-  <xacro:include filename="$(find grizzly_ur10_description/urdf/robotiq_gripper.urdf.xacro" />
+  <xacro:property name="reflect" value="-1" />
+ <xacro:include filename="$(find ur_description)/urdf/gazebo.urdf.xacro" />
+  <xacro:include filename="$(find ur_description)/urdf/ur10_arm.urdf.xacro" />
+  <xacro:include filename="$(find robotiq_s_model_visualization)/cfg/s-model_articulated_macro.urdf.xacro" />
+  <!-- Spawn gripper -->
+  <xacro:s-model_articulated prefix="robotiq_"/>
+  <!-- Add robotiq gripper -->
+  <joint name="ee_joint" type="fixed">
+      <parent link="ee_link"/>
+      <child link="robotiq_palm"/>
+      <origin xyz="0 0 0" rpy="0 0 0" />
+  </joint>
 </robot>

File: grizzly_ur10_description/urdf/ur10_arm.urdf.xacro (robot description, xacro)
@@ -29,8 +29,8 @@
  <xacro:include filename="$(find ur_description)/urdf/gazebo.urdf.xacro" />
   <xacro:include filename="$(find ur_description)/urdf/ur10.urdf.xacro" />
-  <xacro:include filename="$(find robotiq_s_model_visualization)/cfg/s-model_articulated_macro.urdf.xacro" />
   <!-- Spawn arm -->
   <xacro:ur10_robot prefix="ur10_arm_" joint_limited="true"/>
   <!-- <xacro:ur10_robot prefix="" joint_limited="true" /> -->
+  <!-- Join arm -->
   <joint name="grizzly_ur10_joint" type="fixed">
     <parent link="sensor_anchor_link" />
@@ -38,11 +38,3 @@
     <origin xyz="0.65 ${reflect*0.21} 0.03" rpy="0.0 0.0 ${-pi/2}" />
   </joint>
-  <!-- Spawn gripper -->
-  <xacro:s-model_articulated prefix="robotiq_"/>
-  <!-- Add robotiq gripper -->
-  <joint name="ee_joint" type="fixed">
-      <parent link="ee_link"/>
-      <child link="robotiq_palm"/>
-      <origin xyz="0 0 0" rpy="0 0 0" />
-  </joint>
 </robot>

Commit message: Modifying config files.. damn urdf

File: grizzly_ur10_description/urdf/robotiq_gripper.urdf.xacro (robot description, xacro)
@@ -30,10 +30,15 @@
   <xacro:include filename="$(find robotiq_s_model_visualization)/cfg/s-model_articulated_macro.xacro" />
   <!-- Spawn gripper -->
-  <xacro:s-model_articulated prefix="robotiq_"/>
-  <!-- Add robotiq gripper -->
+   <xacro:s-model_articulated prefix="robotiq_"/>
+  <link name="robotiq_gripper_frame_link"/>
+  <joint name="robotiq_gripper_frame_joint" type="fixed">
+      <parent link="ur10_arm_ee_link"/>
+      <child link="robotiq_gripper_frame_link"/>
+      <origin xyz="3.0 0 0" rpy="3.14 0 1.57" />
+  </joint>
   <joint name="ee_joint" type="fixed">
-      <parent link="ur10_arm_ee_link"/>
+      <parent link="robotiq_gripper_frame_link"/>
       <child link="robotiq_palm"/>
-      <origin xyz="0 0 0" rpy="3.14 0 1.57" />
+      <origin xyz="0 0 0" rpy="0 0 0" />
   </joint>
 </robot>

File: grizzly_ur10_description/urdf/test.urdf (robot description, URDF)
Before this commit: robot grizzly_ur10, 31 links, 30 joints
Links:
- removed link robotiq_finger_1_link_0
- removed link robotiq_finger_1_link_1
- removed link robotiq_finger_1_link_2
- removed link robotiq_finger_1_link_3
- removed link robotiq_finger_2_link_0
- removed link robotiq_finger_2_link_1
- removed link robotiq_finger_2_link_2
- removed link robotiq_finger_2_link_3
- removed link robotiq_finger_middle_link_0
- removed link robotiq_finger_middle_link_1
- removed link robotiq_finger_middle_link_2
- removed link robotiq_finger_middle_link_3
- link robotiq_palm: geometry visual mesh filename=package://robotiq_s_model_visualization/meshes/s-model_arti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
Joints:
- removed joint robotiq_finger_1_joint_1
- removed joint robotiq_finger_1_joint_2
- removed joint robotiq_finger_1_joint_3
- removed joint robotiq_finger_2_joint_1
- removed joint robotiq_finger_2_joint_2
- removed joint robotiq_finger_2_joint_3
- removed joint robotiq_finger_middle_joint_1
- removed joint robotiq_finger_middle_joint_2
- removed joint robotiq_finger_middle_joint_3
- removed joint robotiq_palm_finger_1_joint
- removed joint robotiq_palm_finger_2_joint
- removed joint robotiq_palm_finger_middle_joint
- joint ee_joint: origin xyz=0 0 0 rpy=3.14 0 1.57 -> xyz=3.0 0 0 rpy=3.14 0 1.57; type fixed -> continuous

Commit message: Fixed up the urdf config for ee

File: grizzly_ur10_description/urdf/robotiq_gripper.urdf.xacro (robot description, xacro)
@@ -41,15 +41,17 @@
   <!-- Make some joint be the joint between that and the tip link -->
   <!-- ROBOTIQ GRIPPER's TIP LINK = robotiq_finger_middle_link_3 -->
-  <!-- ROBOTIQ GRIPPER's EE_JOINT IS EE_JOINT -->
+  <!-- ROBOTIQ GRIPPER's EE_JOINT IS ur10_arm_ee_joint -->
   <!-- then there should be the tip_link and the joint that connects these.  -->
+  <!-- Chain looks like this:
+   ur10_arm -> ur10_arm_ee_link -> robotiq_palm -> -->
   <link name="robotiq_gripper_tip_frame"/>
   <!-- This connects the robotiq gripper to the ur10 arm -->
-  <joint name="robotiq_gripper_frame_joint" type="fixed">
+  <joint name="ur10_arm_to_gripper_joint" type="fixed">
       <parent link="ur10_arm_ee_link"/>
-      <child link="robotiq_gripper_frame_link"/>
+      <child link="robotiq_palm"/>
       <origin xyz="0 -0.1 0" rpy="1.57 0 1.57" />
   </joint>
   <!-- this is the end effector joint before the tip frame -->
-  <joint name="ee_joint" type="fixed">
+  <joint name="ur10_arm_ee_joint" type="fixed">
       <parent link="robotiq_finger_middle_link_3"/>
       <child link="robotiq_gripper_tip_frame"/>

Commit message: added

File: grizzly_ur10_description/urdf/robotiq_gripper.urdf.xacro (robot description, xacro)
@@ -62,5 +62,5 @@
       <parent link="ur10_arm_ee_link"/>
       <child link="robotiq_palm"/>
-      <origin xyz="0 -0.1 0" rpy="1.57 0 1.57" />
+      <origin xyz="0.01 0 0" rpy="1.57 1.57 0" />
   </joint>
   <!-- this is the end effector joint before the tip frame -->
@@ -68,5 +68,5 @@
       <parent link="robotiq_finger_middle_link_3"/>
       <child link="robotiq_gripper_tip_frame"/>
-      <origin xyz="0.1 0 0" rpy="1.57 0 1.57" />
+      <origin xyz="0 0 0" rpy="0 0 0" />
       <limit lower="-0.25" upper="0.16" effort="100" velocity="100"/>
   </joint>

Commit message: Added proper direct

File: grizzly_ur10_description/urdf/robotiq_gripper.urdf.xacro (robot description, xacro)
@@ -79,5 +79,5 @@
       <origin xyz="0 0 0" rpy="0 0 0"/>
    </xacro:robotiq_hand>
-    <gazebo>
+    <!-- <gazebo>
 	    <plugin name="robotiq_hand_plugin" filename="libRobotiqHandPlugin.so">
 	      <side>left</side>
@@ -85,4 +85,4 @@
 	      <kd_position>0.5</kd_position>
 	     </plugin>
-     </gazebo>
+     </gazebo> -->
 </robot>

File: grizzly_ur10_description/urdf/robotiq_hand.urdf.xacro (robot description, xacro)
@@ -648,5 +648,5 @@
         <visual>
           <geometry>
-            <mesh filename="package://grizzly_ur10_description/meshes/s-model_articulated/visual/palm.STL" />
+            <mesh filename="package://robotiq-s-model_visualization/meshes/s-model_articulated/visual/palm.STL" />
           </geometry>
           <material name="green">

Commit message: Added things

File: grizzly_ur10_description/urdf/robotiq_gripper.urdf.xacro (robot description, xacro)
@@ -84,5 +84,5 @@
      </gazebo>
     <xacro:robotiq_hand prefix="l_" reflect="-1" parent="ur10_arm_ee_link">
-      <origin xyz="0 0 0" rpy="0 0 0"/>
+      <origin xyz="-0.01 0 0" rpy="1.57 0 1.57"/>
    </xacro:robotiq_hand>
 </robot>

Commit message: Fully works in RViz && Gazebo. Robotiq gripper publishing joint states. woot

File: grizzly_ur10_description/urdf/robotiq_gripper.urdf.xacro (robot description, xacro)
@@ -84,5 +84,5 @@
      </gazebo>
     <xacro:robotiq_hand prefix="l_" reflect="-1" parent="ur10_arm_ee_link">
-      <origin xyz="-0.01 0 0" rpy="1.57 0 1.57"/>
+      <origin xyz="-0.01 0 0" rpy="1.57 1.57 0"/>
    </xacro:robotiq_hand>
 </robot>
