Commit message: Appears in gazebo and rviz

File: grizzly_ur10_description/urdf/grizzly_ur10.urdf (robot description, URDF)
Before this commit: robot grizzly_ur10, 18 links, 17 joints
Links:
- removed link ur10_arm_ee_link
- removed link ur10_arm_forearm_link
- removed link ur10_arm_shoulder_link
- removed link ur10_arm_upper_arm_link
- removed link ur10_arm_wrist_1_link
- removed link ur10_arm_wrist_2_link
- removed link ur10_arm_wrist_3_link
- added link ee_link
- added link forearm_link, mass 2.275; collision mesh filename=package://ur_description/meshes/ur10/collision/Forearm.stl; visual mesh filename=package://ur_description/meshes/ur10/visual/Forearm.stl
- added link shoulder_link, mass 3.7; collision mesh filename=package://ur_description/meshes/ur10/collision/Shoulder.stl; visual mesh filename=package://ur_description/meshes/ur10/visual/Shoulder.stl
- added link upper_arm_link, mass 8.393; collision mesh filename=package://ur_description/meshes/ur10/collision/UpperArm.stl; visual mesh filename=package://ur_description/meshes/ur10/visual/UpperArm.stl
- added link wrist_1_link, mass 1.219; collision mesh filename=package://ur_description/meshes/ur10/collision/Wrist1.stl; visual mesh filename=package://ur_description/meshes/ur10/visual/Wrist1.stl
- added link wrist_2_link, mass 1.219; collision mesh filename=package://ur_description/meshes/ur10/collision/Wrist2.stl; visual mesh filename=package://ur_description/meshes/ur10/visual/Wrist2.stl
- added link wrist_3_link, mass 0.1879; collision mesh filename=package://ur_description/meshes/ur10/collision/Wrist3.stl; visual mesh filename=package://ur_description/meshes/ur10/visual/Wrist3.stl
- link back_left_wheel: mass 15 -> 2.63657
- link back_right_wheel: mass 15 -> 2.63657
- link base_footprint: mass None -> 0.0001; geometry visual box size=0.001 0.001 0.001
- link front_axle_link: mass 113 -> 0.45489
- link front_left_wheel: mass 15 -> 2.63657
- link front_right_wheel: mass 15 -> 2.63657
Joints:
- removed joint ur10_arm_ee_fixed_joint
- removed joint ur10_arm_elbow_joint
- removed joint ur10_arm_shoulder_lift_joint
- removed joint ur10_arm_shoulder_pan_joint
- removed joint ur10_arm_wrist_1_joint
- removed joint ur10_arm_wrist_2_joint
- removed joint ur10_arm_wrist_3_joint
- added joint ee_fixed_joint: type fixed, parent wrist_3_link, child ee_link, origin xyz=0.0 0.0857 0.0 rpy=0.0 0.0 1.570796325
- added joint elbow_joint: type revolute, parent upper_arm_link, child forearm_link, origin xyz=0.0 -0.12817 0.60186 rpy=0.0 0.0 0.0, axis 0.0 1.0 0.0, limit lower=-6.2831853 upper=6.2831853 effort=150.0 velocity=3.14159265
- added joint shoulder_lift_joint: type revolute, parent shoulder_link, child upper_arm_link, origin xyz=0.0 0.1704 0.0 rpy=0.0 1.570796325 0.0, axis 0.0 1.0 0.0, limit lower=-6.2831853 upper=6.2831853 effort=10.0 velocity=3.14159265
- added joint shoulder_pan_joint: type revolute, parent ur10_arm_base_link, child shoulder_link, origin xyz=0.0 0.0 0.128 rpy=0.0 0.0 0.0, axis 0.0 0.0 1.0, limit lower=-6.2831853 upper=6.2831853 effort=330.0 velocity=2.16
- added joint wrist_1_joint: type revolute, parent forearm_link, child wrist_1_link, origin xyz=0.0 0.0 0.56415 rpy=0.0 1.570796325 0.0, axis 0.0 1.0 0.0, limit lower=-6.2831853 upper=6.2831853 effort=54.0 velocity=3.14159265
- added joint wrist_2_joint: type revolute, parent wrist_1_link, child wrist_2_link, origin xyz=0.0 0.11279 0.0 rpy=0.0 0.0 0.0, axis 0.0 0.0 1.0, limit lower=-6.2831853 upper=6.2831853 effort=54.0 velocity=3.14159265
- added joint wrist_3_joint: type revolute, parent wrist_2_link, child wrist_3_link, origin xyz=0.0 0.0 0.11279 rpy=0.0 0.0 0.0, axis 0.0 1.0 0.0, limit lower=-6.2831853 upper=6.2831853 effort=54.0 velocity=3.14159265

Commit message: Removed disable collisions

File: grizzly_ur10_description/urdf/grizzly_ur10.urdf (robot description, URDF)
Before this commit: robot grizzly_ur10, 18 links, 17 joints
Links:
- link back_left_wheel: mass 2.63657 -> 15
- link back_right_wheel: mass 2.63657 -> 15
- link base_footprint: mass 0.0001 -> None; geometry 
- link front_axle_link: mass 0.45489 -> 113
- link front_left_wheel: mass 2.63657 -> 15
- link front_right_wheel: mass 2.63657 -> 15

Commit message: Added ur10_arm_ prefix

File: grizzly_ur10_description/urdf/grizzly_ur10.urdf (robot description, URDF)
Before this commit: robot grizzly_ur10, 18 links, 17 joints
Links:
- removed link ur10_arm_base_link
- link base_link: geometry collision mesh filename=package://ur_description/meshes/ur10/collision/base.stl; visual mesh filename=package://ur_description/meshes/ur10/visual/Base.dae
- link ee_link: geometry collision box size=0.01 0.01 0.01
- link forearm_link: mass 2.275 -> 3.87; geometry collision mesh filename=package://ur_description/meshes/ur10/collision/forearm.stl; visual mesh filename=package://ur_description/meshes/ur10/visual/Forearm.dae
- link shoulder_link: mass 3.7 -> 7.778; geometry collision mesh filename=package://ur_description/meshes/ur10/collision/shoulder.stl; visual mesh filename=package://ur_description/meshes/ur10/visual/Shoulder.dae
- link upper_arm_link: mass 8.393 -> 12.93; geometry collision mesh filename=package://ur_description/meshes/ur10/collision/upper_arm.stl; visual mesh filename=package://ur_description/meshes/ur10/visual/UpperArm.dae
- link wrist_1_link: mass 1.219 -> 1.96; geometry collision mesh filename=package://ur_description/meshes/ur10/collision/wrist_1.stl; visual mesh filename=package://ur_description/meshes/ur10/visual/Wrist1.dae
- link wrist_2_link: mass 1.219 -> 1.96; geometry collision mesh filename=package://ur_description/meshes/ur10/collision/wrist_2.stl; visual mesh filename=package://ur_description/meshes/ur10/visual/Wrist2.dae
- link wrist_3_link: mass 0.1879 -> 0.202; geometry collision mesh filename=package://ur_description/meshes/ur10/collision/wrist_3.stl; visual mesh filename=package://ur_description/meshes/ur10/visual/Wrist3.dae
Joints:
- joint ee_fixed_joint: origin xyz=0.0 0.0857 0.0 rpy=0.0 0.0 1.570796325 -> xyz=0.0 0.0922 0.0 rpy=0.0 0.0 1.570796325
- joint elbow_joint: axis 0.0 1.0 0.0 -> 0 1 0; limit lower=-6.2831853 upper=6.2831853 effort=150.0 velocity=3.14159265 -> lower=-3.14159265 upper=3.14159265 effort=150.0 velocity=3.15; origin xyz=0.0 -0.12817 0.60186 rpy=0.0 0.0 0.0 -> xyz=0.0 -0.1719 0.612 rpy=0.0 0.0 0.0
- joint shoulder_lift_joint: axis 0.0 1.0 0.0 -> 0 1 0; limit lower=-6.2831853 upper=6.2831853 effort=10.0 velocity=3.14159265 -> lower=-3.14159265 upper=3.14159265 effort=330.0 velocity=2.16; origin xyz=0.0 0.1704 0.0 rpy=0.0 1.570796325 0.0 -> xyz=0.0 0.220941 0.0 rpy=0.0 1.570796325 0.0
- joint shoulder_pan_joint: axis 0.0 0.0 1.0 -> 0 0 1; limit lower=-6.2831853 upper=6.2831853 effort=330.0 velocity=2.16 -> lower=-3.14159265 upper=3.14159265 effort=330.0 velocity=2.16; origin xyz=0.0 0.0 0.128 rpy=0.0 0.0 0.0 -> xyz=0.0 0.0 0.1273 rpy=0.0 0.0 0.0; parent ur10_arm_base_link -> base_link
- joint wrist_1_joint: axis 0.0 1.0 0.0 -> 0 1 0; limit lower=-6.2831853 upper=6.2831853 effort=54.0 velocity=3.14159265 -> lower=-3.14159265 upper=3.14159265 effort=54.0 velocity=3.2; origin xyz=0.0 0.0 0.56415 rpy=0.0 1.570796325 0.0 -> xyz=0.0 0.0 0.5723 rpy=0.0 1.570796325 0.0
- joint wrist_2_joint: axis 0.0 0.0 1.0 -> 0 0 1; limit lower=-6.2831853 upper=6.2831853 effort=54.0 velocity=3.14159265 -> lower=-3.14159265 upper=3.14159265 effort=54.0 velocity=3.2; origin xyz=0.0 0.11279 0.0 rpy=0.0 0.0 0.0 -> xyz=0.0 0.1149 0.0 rpy=0.0 0.0 0.0
- joint wrist_3_joint: axis 0.0 1.0 0.0 -> 0 1 0; limit lower=-6.2831853 upper=6.2831853 effort=54.0 velocity=3.14159265 -> lower=-3.14159265 upper=3.14159265 effort=54.0 velocity=3.2; origin xyz=0.0 0.0 0.11279 rpy=0.0 0.0 0.0 -> xyz=0.0 0.0 0.1157 rpy=0.0 0.0 0.0

File: grizzly_ur10_description/urdf/manipulator.urdf.xacro (robot description, xacro)
@@ -30,5 +30,5 @@
   <xacro:include filename="$(find ur_description)/urdf/ur10.urdf.xacro" />
   <!-- Spawn arm -->
-  <xacro:ur10_robot prefix="" joint_limited="true"/>
+  <xacro:ur10_robot prefix="ur10_arm_" joint_limited="true"/>
   <!-- <xacro:ur10_robot prefix="" joint_limited="true" /> -->
   <joint name="grizzly_ur10_joint" type="fixed">

Commit message: modified all joint names in moveit config

File: grizzly_ur10_description/urdf/grizzly_ur10.urdf (robot description, URDF)
Before this commit: robot grizzly_ur10, 17 links, 17 joints
Links:
- removed link ee_link
- removed link forearm_link
- removed link shoulder_link
- removed link upper_arm_link
- removed link wrist_1_link
- removed link wrist_2_link
- removed link wrist_3_link
- added link ur10_arm_base_link, mass 4.0; collision mesh filename=package://ur_description/meshes/ur10/collision/base.stl; visual mesh filename=package://ur_description/meshes/ur10/visual/Base.dae
- added link ur10_arm_ee_link; collision box size=0.01 0.01 0.01
- added link ur10_arm_forearm_link, mass 3.87; collision mesh filename=package://ur_description/meshes/ur10/collision/forearm.stl; visual mesh filename=package://ur_description/meshes/ur10/visual/Forearm.dae
- added link ur10_arm_shoulder_link, mass 7.778; collision mesh filename=package://ur_description/meshes/ur10/collision/shoulder.stl; visual mesh filename=package://ur_description/meshes/ur10/visual/Shoulder.dae
- added link ur10_arm_upper_arm_link, mass 12.93; collision mesh filename=package://ur_description/meshes/ur10/collision/upper_arm.stl; visual mesh filename=package://ur_description/meshes/ur10/visual/UpperArm.dae
- added link ur10_arm_wrist_1_link, mass 1.96; collision mesh filename=package://ur_description/meshes/ur10/collision/wrist_1.stl; visual mesh filename=package://ur_description/meshes/ur10/visual/Wrist1.dae
- added link ur10_arm_wrist_2_link, mass 1.96; collision mesh filename=package://ur_description/meshes/ur10/collision/wrist_2.stl; visual mesh filename=package://ur_description/meshes/ur10/visual/Wrist2.dae
- added link ur10_arm_wrist_3_link, mass 0.202; collision mesh filename=package://ur_description/meshes/ur10/collision/wrist_3.stl; visual mesh filename=package://ur_description/meshes/ur10/visual/Wrist3.dae
- link base_link: geometry collision box size=0.708 0.3 1.826; visual mesh filename=package://grizzly_description/meshes/base_link.stl
Joints:
- removed joint ee_fixed_joint
- removed joint elbow_joint
- removed joint shoulder_lift_joint
- removed joint shoulder_pan_joint
- removed joint wrist_1_joint
- removed joint wrist_2_joint
- removed joint wrist_3_joint
- added joint ur10_arm_ee_fixed_joint: type fixed, parent ur10_arm_wrist_3_link, child ur10_arm_ee_link, origin xyz=0.0 0.0922 0.0 rpy=0.0 0.0 1.570796325
- added joint ur10_arm_elbow_joint: type revolute, parent ur10_arm_upper_arm_link, child ur10_arm_forearm_link, origin xyz=0.0 -0.1719 0.612 rpy=0.0 0.0 0.0, axis 0 1 0, limit lower=-3.14159265 upper=3.14159265 effort=150.0 velocity=3.15
- added joint ur10_arm_shoulder_lift_joint: type revolute, parent ur10_arm_shoulder_link, child ur10_arm_upper_arm_link, origin xyz=0.0 0.220941 0.0 rpy=0.0 1.570796325 0.0, axis 0 1 0, limit lower=-3.14159265 upper=3.14159265 effort=330.0 velocity=2.16
- added joint ur10_arm_shoulder_pan_joint: type revolute, parent ur10_arm_base_link, child ur10_arm_shoulder_link, origin xyz=0.0 0.0 0.1273 rpy=0.0 0.0 0.0, axis 0 0 1, limit lower=-3.14159265 upper=3.14159265 effort=330.0 velocity=2.16
- added joint ur10_arm_wrist_1_joint: type revolute, parent ur10_arm_forearm_link, child ur10_arm_wrist_1_link, origin xyz=0.0 0.0 0.5723 rpy=0.0 1.570796325 0.0, axis 0 1 0, limit lower=-3.14159265 upper=3.14159265 effort=54.0 velocity=3.2
- added joint ur10_arm_wrist_2_joint: type revolute, parent ur10_arm_wrist_1_link, child ur10_arm_wrist_2_link, origin xyz=0.0 0.1149 0.0 rpy=0.0 0.0 0.0, axis 0 0 1, limit lower=-3.14159265 upper=3.14159265 effort=54.0 velocity=3.2
- added joint ur10_arm_wrist_3_joint: type revolute, parent ur10_arm_wrist_2_link, child ur10_arm_wrist_3_link, origin xyz=0.0 0.0 0.1157 rpy=0.0 0.0 0.0, axis 0 1 0, limit lower=-3.14159265 upper=3.14159265 effort=54.0 velocity=3.2

Commit message: Added robotiq_gripper moveit configs

File: grizzly_ur10_description/urdf/grizzly_ur10.urdf (robot description, URDF)
Before this commit: robot grizzly_ur10, 31 links, 30 joints
Joints:
- joint ee_joint: origin xyz=0 0 0 rpy=1.57 0.78 0.78 -> xyz=0 0 0 rpy=3.14 0 1.57

Commit message: Changed robotiq description to use mesh

File: grizzly_ur10_description/urdf/grizzly_ur10.urdf (robot description, URDF)
Before this commit: robot grizzly_ur10, 31 links, 30 joints
Links:
- removed link robotiq_finger_1_link_0
- removed link robotiq_finger_1_link_1
- removed link robotiq_finger_1_link_2
- removed link robotiq_finger_1_link_3
- removed link robotiq_finger_2_link_0
- removed link robotiq_finger_2_link_1
- removed link robotiq_finger_2_link_2
- removed link robotiq_finger_2_link_3
- removed link robotiq_finger_middle_link_0
- removed link robotiq_finger_middle_link_1
- removed link robotiq_finger_middle_link_2
- removed link robotiq_finger_middle_link_3
- added link robotiq_finger_1; collision mesh filename=package://robotiq_s_model_visualization/meshes/s-model/coll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; visual mesh filename=package://robotiq_s_model_visualization/meshes/s-model/visu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
- added link robotiq_finger_2; collision mesh filename=package://robotiq_s_model_visualization/meshes/s-model/coll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; visual mesh filename=package://robotiq_s_model_visualization/meshes/s-model/visu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
- added link robotiq_finger_3; collision mesh filename=package://robotiq_s_model_visualization/meshes/s-model/coll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; visual mesh filename=package://robotiq_s_model_visualization/meshes/s-model/visu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
- added link robotiq_gripper_frame_link
- link robotiq_palm: geometry collision mesh filename=package://robotiq_s_model_visualization/meshes/s-model/coll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; visual mesh filename=package://robotiq_s_model_visualization/meshes/s-model/visu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
Joints:
- removed joint robotiq_finger_1_joint_1
- removed joint robotiq_finger_1_joint_2
- removed joint robotiq_finger_1_joint_3
- removed joint robotiq_finger_2_joint_1
- removed joint robotiq_finger_2_joint_2
- removed joint robotiq_finger_2_joint_3
- removed joint robotiq_finger_middle_joint_1
- removed joint robotiq_finger_middle_joint_2
- removed joint robotiq_finger_middle_joint_3
- removed joint robotiq_palm_finger_1_joint
- removed joint robotiq_palm_finger_2_joint
- removed joint robotiq_palm_finger_middle_joint
- added joint robotiq_gripper_frame_joint: type fixed, parent ur10_arm_ee_link, child robotiq_gripper_frame_link, origin xyz=0 0 0 rpy=0 0 0
- added joint robotiq_joint_1: type fixed, parent robotiq_palm, child robotiq_finger_1, origin xyz=0 0 0 rpy=0 0 0
- added joint robotiq_joint_2: type fixed, parent robotiq_palm, child robotiq_finger_2, origin xyz=0 0 0 rpy=0 0 0
- added joint robotiq_joint_3: type fixed, parent robotiq_palm, child robotiq_finger_3, origin xyz=0 0 0 rpy=0 0 0
- joint ee_joint: origin xyz=0 0 0 rpy=3.14 0 1.57 -> xyz=0.1 0 0 rpy=1.57 0 1.57; parent ur10_arm_ee_link -> robotiq_gripper_frame_link

File: grizzly_ur10_description/urdf/robotiq_gripper.urdf.xacro (robot description, xacro)
@@ -28,17 +28,18 @@
   <xacro:property name="reflect" value="-1" />
  <xacro:include filename="$(find ur_description)/urdf/gazebo.urdf.xacro" />
-  <xacro:include filename="$(find robotiq_s_model_visualization)/cfg/s-model_articulated_macro.xacro" />
+  <!-- <xacro:include filename="$(find robotiq_s_model_visualization)/cfg/s-model_articulated_macro.xacro" /> -->
+   <xacro:include filename="$(find robotiq_s_model_visualization)/cfg/s-model_mesh_macro.xacro"/>
   <!-- Spawn gripper -->
-   <xacro:s-model_articulated prefix="robotiq_"/>
+   <xacro:s-model_mesh prefix="robotiq_"/>
   <link name="robotiq_gripper_frame_link"/>
   <joint name="robotiq_gripper_frame_joint" type="fixed">
       <parent link="ur10_arm_ee_link"/>
       <child link="robotiq_gripper_frame_link"/>
-      <origin xyz="3.0 0 0" rpy="3.14 0 1.57" />
+      <origin xyz="0 0 0" rpy="0 0 0" />
   </joint>
   <joint name="ee_joint" type="fixed">
       <parent link="robotiq_gripper_frame_link"/>
       <child link="robotiq_palm"/>
-      <origin xyz="0 0 0" rpy="0 0 0" />
+      <origin xyz="0.1 0 0" rpy="1.57 0 1.57" />
   </joint>
 </robot>

File: grizzly_ur10_description/urdf/urdf.urdf (robot description, URDF)
Before this commit: robot grizzly_ur10, 19 links, 18 joints
Links:
- added link robotiq_gripper_frame_link
- link robotiq_palm: geometry collision mesh filename=package://robotiq_s_model_visualization/meshes/s-model_arti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; visual mesh filename=package://robotiq_s_model_visualization/meshes/s-model_arti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
Joints:
- added joint robotiq_gripper_frame_joint: type fixed, parent ur10_arm_ee_link, child robotiq_gripper_frame_link, origin xyz=3.0 0 0 rpy=3.14 0 1.57
- joint ee_joint: origin xyz=3.0 0 0 rpy=3.14 0 1.57 -> xyz=0 0 0 rpy=0 0 0; parent ur10_arm_ee_link -> robotiq_gripper_frame_link; type continuous -> fixed

Commit message: aoshgsuhgUHDUH

File: grizzly_ur10_description/urdf/grizzly_ur10.urdf (robot description, URDF)
Before this commit: robot grizzly_ur10, 32 links, 31 joints
Links:
- link robotiq_finger_1_link_0: geometry visual mesh filename=package://robotiq_s_model_visualization/meshes/s-model_arti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
- link robotiq_finger_1_link_1: geometry visual mesh filename=package://robotiq_s_model_visualization/meshes/s-model_arti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
- link robotiq_finger_1_link_2: geometry visual mesh filename=package://robotiq_s_model_visualization/meshes/s-model_arti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
- link robotiq_finger_1_link_3: geometry visual mesh filename=package://robotiq_s_model_visualization/meshes/s-model_arti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
- link robotiq_finger_2_link_0: geometry visual mesh filename=package://robotiq_s_model_visualization/meshes/s-model_arti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
- link robotiq_finger_2_link_1: geometry visual mesh filename=package://robotiq_s_model_visualization/meshes/s-model_arti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
- link robotiq_finger_2_link_2: geometry visual mesh filename=package://robotiq_s_model_visualization/meshes/s-model_arti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
- link robotiq_finger_2_link_3: geometry visual mesh filename=package://robotiq_s_model_visualization/meshes/s-model_arti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
- link robotiq_finger_middle_link_0: geometry visual mesh filename=package://robotiq_s_model_visualization/meshes/s-model_arti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
- link robotiq_finger_middle_link_1: geometry visual mesh filename=package://robotiq_s_model_visualization/meshes/s-model_arti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
- link robotiq_finger_middle_link_2: geometry visual mesh filename=package://robotiq_s_model_visualization/meshes/s-model_arti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
- link robotiq_finger_middle_link_3: geometry visual mesh filename=package://robotiq_s_model_visualization/meshes/s-model_arti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
- link robotiq_palm: geometry visual mesh filename=package://robotiq_s_model_visualization/meshes/s-model_arti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

Commit message: Updated

File: grizzly_ur10_description/urdf/grizzly_ur10.urdf (robot description, URDF)
Before this commit: robot grizzly_ur10, 32 links, 31 joints
Links:
- removed link robotiq_finger_1_link_0
- removed link robotiq_finger_1_link_1
- removed link robotiq_finger_1_link_2
- removed link robotiq_finger_1_link_3
- removed link robotiq_finger_2_link_0
- removed link robotiq_finger_2_link_1
- removed link robotiq_finger_2_link_2
- removed link robotiq_finger_2_link_3
- removed link robotiq_finger_middle_link_0
- removed link robotiq_finger_middle_link_1
- removed link robotiq_finger_middle_link_2
- removed link robotiq_finger_middle_link_3
- link robotiq_palm: geometry collision mesh filename=package://robotiq_s_model_visualization/meshes/s-model_arti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; visual mesh filename=package://robotiq_s_model_visualization/meshes/s-model_arti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
Joints:
- removed joint robotiq_finger_1_joint_1
- removed joint robotiq_finger_1_joint_2
- removed joint robotiq_finger_1_joint_3
- removed joint robotiq_finger_2_joint_1
- removed joint robotiq_finger_2_joint_2
- removed joint robotiq_finger_2_joint_3
- removed joint robotiq_finger_middle_joint_1
- removed joint robotiq_finger_middle_joint_2
- removed joint robotiq_finger_middle_joint_3
- removed joint robotiq_palm_finger_1_joint
- removed joint robotiq_palm_finger_2_joint
- removed joint robotiq_palm_finger_middle_joint
