Commit message: Added properurdf orientation for gripper

File: grizzly_ur10_description/urdf/grizzly_ur10.urdf (robot description, URDF)
Before this commit: robot grizzly_ur10, 20 links, 19 joints
Links:
- added link robotiq_finger_1_link_0, mass 0.05; collision mesh filename=package://robotiq_s_model_visualization/meshes/s-model_arti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; visual mesh filename=package://robotiq_s_model_visualization/meshes/s-model_arti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
- added link robotiq_finger_1_link_1, mass 0.15; collision mesh filename=package://robotiq_s_model_visualization/meshes/s-model_arti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; visual mesh filename=package://robotiq_s_model_visualization/meshes/s-model_arti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
- added link robotiq_finger_1_link_2, mass 0.15; collision mesh filename=package://robotiq_s_model_visualization/meshes/s-model_arti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; visual mesh filename=package://robotiq_s_model_visualization/meshes/s-model_arti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
- added link robotiq_finger_1_link_3, mass 0.05; collision mesh filename=package://robotiq_s_model_visualization/meshes/s-model_arti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; visual mesh filename=package://robotiq_s_model_visualization/meshes/s-model_arti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
- added link robotiq_finger_2_link_0, mass 0.05; collision mesh filename=package://robotiq_s_model_visualization/meshes/s-model_arti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; visual mesh filename=package://robotiq_s_model_visualization/meshes/s-model_arti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
- added link robotiq_finger_2_link_1, mass 0.15; collision mesh filename=package://robotiq_s_model_visualization/meshes/s-model_arti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; visual mesh filename=package://robotiq_s_model_visualization/meshes/s-model_arti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
- added link robotiq_finger_2_link_2, mass 0.15; collision mesh filename=package://robotiq_s_model_visualization/meshes/s-model_arti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; visual mesh filename=package://robotiq_s_model_visualization/meshes/s-model_arti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
- added link robotiq_finger_2_link_3, mass 0.05; collision mesh filename=package://robotiq_s_model_visualization/meshes/s-model_arti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; visual mesh filename=package://robotiq_s_model_visualization/meshes/s-model_arti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
- added link robotiq_finger_middle_link_0, mass 0.05; collision mesh filename=package://robotiq_s_model_visualization/meshes/s-model_arti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; visual mesh filename=package://robotiq_s_model_visualization/meshes/s-model_arti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
- added link robotiq_finger_middle_link_1, mass 0.15; collision mesh filename=package://robotiq_s_model_visualization/meshes/s-model_arti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; visual mesh filename=package://robotiq_s_model_visualization/meshes/s-model_arti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
- added link robotiq_finger_middle_link_2, mass 0.15; collision mesh filename=package://robotiq_s_model_visualization/meshes/s-model_arti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; visual mesh filename=package://robotiq_s_model_visualization/meshes/s-model_arti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
- added link robotiq_finger_middle_link_3, mass 0.05; collision mesh filename=package://robotiq_s_model_visualization/meshes/s-model_arti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; visual mesh filename=package://robotiq_s_model_visualization/meshes/s-model_arti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
Joints:
- added joint robotiq_finger_1_joint_1: type revolute, parent robotiq_finger_1_link_0, child robotiq_finger_1_link_1, origin xyz=0.020 0 0 rpy=0 0 0, axis 0 0 1, limit lower=0 upper=3.1416 effort=100 velocity=100
- added joint robotiq_finger_1_joint_2: type revolute, parent robotiq_finger_1_link_1, child robotiq_finger_1_link_2, origin xyz=0.050 -.028 0 rpy=0 0 -0.52, axis 0 0 1, limit lower=0 upper=3.1416 effort=100 velocity=100
- added joint robotiq_finger_1_joint_3: type revolute, parent robotiq_finger_1_link_2, child robotiq_finger_1_link_3, origin xyz=0.039 0 0 rpy=0 0 0, axis 0 0 1, limit lower=0 upper=3.1416 effort=100 velocity=100
- added joint robotiq_finger_2_joint_1: type revolute, parent robotiq_finger_2_link_0, child robotiq_finger_2_link_1, origin xyz=0.020 0 0 rpy=0 0 0, axis 0 0 1, limit lower=0 upper=3.1416 effort=100 velocity=100
- added joint robotiq_finger_2_joint_2: type revolute, parent robotiq_finger_2_link_1, child robotiq_finger_2_link_2, origin xyz=0.050 -.028 0 rpy=0 0 -0.52, axis 0 0 1, limit lower=0 upper=3.1416 effort=100 velocity=100
- added joint robotiq_finger_2_joint_3: type revolute, parent robotiq_finger_2_link_2, child robotiq_finger_2_link_3, origin xyz=0.039 0 0 rpy=0 0 0, axis 0 0 1, limit lower=0 upper=3.1416 effort=100 velocity=100
- added joint robotiq_finger_middle_joint_1: type revolute, parent robotiq_finger_middle_link_0, child robotiq_finger_middle_link_1, origin xyz=0.020 0 0 rpy=0 0 0, axis 0 0 1, limit lower=0 upper=3.1416 effort=100 velocity=100
- added joint robotiq_finger_middle_joint_2: type revolute, parent robotiq_finger_middle_link_1, child robotiq_finger_middle_link_2, origin xyz=0.050 -.028 0 rpy=0 0 -0.52, axis 0 0 1, limit lower=0 upper=3.1416 effort=100 velocity=100
- added joint robotiq_finger_middle_joint_3: type revolute, parent robotiq_finger_middle_link_2, child robotiq_finger_middle_link_3, origin xyz=0.039 0 0 rpy=0 0 0, axis 0 0 1, limit lower=0 upper=3.1416 effort=100 velocity=100
- added joint robotiq_palm_finger_1_joint: type revolute, parent robotiq_palm, child robotiq_finger_1_link_0, origin xyz=-0.0455 0.0214 0.036 rpy=0 3.1416 -1.57, axis 0 1 0, limit lower=-0.16 upper=0.25 effort=100 velocity=100
- added joint robotiq_palm_finger_2_joint: type revolute, parent robotiq_palm, child robotiq_finger_2_link_0, origin xyz=-0.0455 0.0214 -0.036 rpy=0 3.1416 -1.57, axis 0 1 0, limit lower=-0.25 upper=0.16 effort=100 velocity=100
- added joint robotiq_palm_finger_middle_joint: type fixed, parent robotiq_palm, child robotiq_finger_middle_link_0, origin xyz=0.0455 0.0214 0 rpy=0 0 1.57, axis 0 0 1

File: grizzly_ur10_description/urdf/robotiq_gripper.urdf.xacro (robot description, xacro)
@@ -27,6 +27,5 @@
 <robot xmlns:xacro="http://ros.org/wiki/xacro" name="grizzly_ur10">
   <xacro:property name="reflect" value="-1" />
- <xacro:include filename="$(find ur_description)/urdf/gazebo.urdf.xacro" />
-  <!-- <xacro:include filename="$(find robotiq_s_model_visualization)/cfg/s-model_articulated_macro.xacro" /> -->
+   <xacro:include filename="$(find ur_description)/urdf/gazebo.urdf.xacro" />
    <xacro:include filename="$(find robotiq_s_model_visualization)/cfg/s-model_articulated_macro.xacro"/>
   <!-- Spawn gripper -->
@@ -36,5 +35,5 @@
       <parent link="ur10_arm_ee_link"/>
       <child link="robotiq_gripper_frame_link"/>
-      <origin xyz="0 0 0" rpy="0 0 0" />
+      <origin xyz="0 -0.1 0" rpy="1.57 0 1.57" />
   </joint>
   <joint name="ee_joint" type="fixed">

Commit message: Updated

File: grizzly_ur10_description/urdf/grizzly_ur10.urdf (robot description, URDF)
Before this commit: robot grizzly_ur10, 32 links, 31 joints
Joints:
- joint robotiq_gripper_frame_joint: origin xyz=0 0 0 rpy=0 0 0 -> xyz=0 -0.1 0 rpy=1.57 0 1.57

Commit message: updated

File: grizzly_ur10_description/urdf/grizzly_ur10.urdf (robot description, URDF)
Before this commit: robot grizzly_ur10, 33 links, 32 joints
Links:
- added link grizzly_ur10_hokuyo_link, mass 0.001
- added link grizzly_ur10_kinect_optical_frame
- link grizzly_ur10_kinect_frame: mass None -> 0.1; geometry collision mesh filename=package://pr2_description/meshes/sensors/kinect_v0/kinect.d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 scale=0.001 0.001 0.001; visual mesh filename=package://pr2_description/meshes/sensors/kinect_v0/kinect.d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 scale=0.001 0.001 0.001
Joints:
- added joint grizzly_ur10_hokuyo_joint: type fixed, parent sensor_anchor_link, child grizzly_ur10_hokuyo_link, origin xyz=1.0 0 -0.1 rpy=0 0 0, axis 0 1 0
- added joint grizzly_ur10_kinect_optical_joint: type fixed, parent grizzly_ur10_kinect_frame, child grizzly_ur10_kinect_optical_frame, origin xyz=0.0            0.0         0.0 rpy=-1.57079632679 0.0 -1.57079632679
- joint grizzly_ur10_kinect_frame_joint: origin xyz=0 0 0 rpy=0 0 0 -> xyz=0.5 0 0.4 rpy=0 0.349065850399 0; type None -> fixed

Commit message: Buncha bug fixes

File: grizzly_ur10_description/urdf/grizzly_ur10.urdf (robot description, URDF)
Before this commit: robot grizzly_ur10, 35 links, 34 joints
Links:
- link robotiq_palm: mass None -> 1.3

File: grizzly_ur10_description/urdf/robotiq_gripper.urdf.xacro (robot description, xacro)
@@ -29,4 +29,6 @@
    <xacro:include filename="$(find ur_description)/urdf/gazebo.urdf.xacro" />
    <xacro:include filename="$(find robotiq_s_model_visualization)/cfg/s-model_articulated_macro.xacro"/>
+   <!-- Transmission for robotiq gripper so that it can use ROS control -->
+   <xacro:include filename="$(find grizzly_ur10_description)/urdf/s-model_articulated.transmission.xacro" />
   <!-- Spawn gripper -->
    <xacro:s-model_articulated prefix="robotiq_"/>
@@ -82,3 +84,5 @@
       <selfCollide>true</selfCollide>
   </gazebo>
+    <!-- Instantiate transmission file -->
+    <xacro:robotiq_gripper_transmission prefix="" />
 </robot>

Commit message: ok

File: grizzly_ur10_description/urdf/grizzly_ur10.urdf (robot description, URDF)
Before this commit: robot grizzly_ur10, 35 links, 34 joints
Joints:
- joint robotiq_palm_finger_middle_joint: limit (none) -> lower=-0.25 upper=0.16 effort=100 velocity=100; type fixed -> revolute

File: grizzly_ur10_description/urdf/robotiq_gripper.urdf.xacro (robot description, xacro)
@@ -38,6 +38,11 @@
   <!-- Note: the gripper_action_controller and MoveIt require a specific structure of the URDF so that this will work.
    end_of_robotiq_finger_tip -> joint -> tip_link -> ee_joint -> tip_frame -->
-  <!-- End of robotiq gripper = robotiq_palm_finger -->
-  <link name="robotiq_gripper_frame_link"/>
+  <!-- End of robotiq gripper = robotiq_finger_middle_link_3 -->
+  <!-- Make some joint be the joint between that and the tip link -->
+  <!-- ROBOTIQ GRIPPER's TIP LINK = robotiq_finger_middle_link_3 -->
+  <!-- ROBOTIQ GRIPPER's EE_JOINT IS EE_JOINT -->
+  <!-- then there should be the tip_link and the joint that connects these.  -->
+  <link name="robotiq_gripper_tip_frame"/>
+  <!-- This connects the robotiq gripper to the ur10 arm -->
   <joint name="robotiq_gripper_frame_joint" type="fixed">
       <parent link="ur10_arm_ee_link"/>
@@ -45,7 +50,8 @@
       <origin xyz="0 -0.1 0" rpy="1.57 0 1.57" />
   </joint>
+  <!-- this is the end effector joint before the tip frame -->
   <joint name="ee_joint" type="fixed">
-      <parent link="robotiq_gripper_frame_link"/>
-      <child link="robotiq_palm"/>
+      <parent link="robotiq_finger_middle_link_3"/>
+      <child link="robotiq_gripper_tip_frame"/>
       <origin xyz="0.1 0 0" rpy="1.57 0 1.57" />
   </joint>

Commit message: Fixing git?

File: grizzly_ur10_description/urdf/grizzly_ur10.urdf (robot description, URDF)
Before this commit: robot grizzly_ur10, 18 links, 17 joints
Links:
- added link grizzly_ur10_hokuyo_link, mass 0.001
- added link grizzly_ur10_kinect_frame, mass 0.1; collision mesh filename=package://pr2_description/meshes/sensors/kinect_v0/kinect.d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 scale=0.001 0.001 0.001; visual mesh filename=package://pr2_description/meshes/sensors/kinect_v0/kinect.d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 scale=0.001 0.001 0.001
- added link grizzly_ur10_kinect_optical_frame
- added link robotiq_finger_1_link_0, mass 0.05; collision mesh filename=package://robotiq_s_model_visualization/meshes/s-model_arti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; visual mesh filename=package://robotiq_s_model_visualization/meshes/s-model_arti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
- added link robotiq_finger_1_link_1, mass 0.15; collision mesh filename=package://robotiq_s_model_visualization/meshes/s-model_arti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; visual mesh filename=package://robotiq_s_model_visualization/meshes/s-model_arti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
- added link robotiq_finger_1_link_2, mass 0.15; collision mesh filename=package://robotiq_s_model_visualization/meshes/s-model_arti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; visual mesh filename=package://robotiq_s_model_visualization/meshes/s-model_arti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
- added link robotiq_finger_1_link_3, mass 0.05; collision mesh filename=package://robotiq_s_model_visualization/meshes/s-model_arti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; visual mesh filename=package://robotiq_s_model_visualization/meshes/s-model_arti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
- added link robotiq_finger_2_link_0, mass 0.05; collision mesh filename=package://robotiq_s_model_visualization/meshes/s-model_arti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; visual mesh filename=package://robotiq_s_model_visualization/meshes/s-model_arti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
- added link robotiq_finger_2_link_1, mass 0.15; collision mesh filename=package://robotiq_s_model_visualization/meshes/s-model_arti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; visual mesh filename=package://robotiq_s_model_visualization/meshes/s-model_arti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
- added link robotiq_finger_2_link_2, mass 0.15; collision mesh filename=package://robotiq_s_model_visualization/meshes/s-model_arti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; visual mesh filename=package://robotiq_s_model_visualization/meshes/s-model_arti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
- added link robotiq_finger_2_link_3, mass 0.05; collision mesh filename=package://robotiq_s_model_visualization/meshes/s-model_arti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; visual mesh filename=package://robotiq_s_model_visualization/meshes/s-model_arti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
- added link robotiq_finger_middle_link_0, mass 0.05; collision mesh filename=package://robotiq_s_model_visualization/meshes/s-model_arti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; visual mesh filename=package://robotiq_s_model_visualization/meshes/s-model_arti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
- added link robotiq_finger_middle_link_1, mass 0.15; collision mesh filename=package://robotiq_s_model_visualization/meshes/s-model_arti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; visual mesh filename=package://robotiq_s_model_visualization/meshes/s-model_arti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
- added link robotiq_finger_middle_link_2, mass 0.15; collision mesh filename=package://robotiq_s_model_visualization/meshes/s-model_arti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; visual mesh filename=package://robotiq_s_model_visualization/meshes/s-model_arti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
- added link robotiq_finger_middle_link_3, mass 0.05; collision mesh filename=package://robotiq_s_model_visualization/meshes/s-model_arti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; visual mesh filename=package://robotiq_s_model_visualization/meshes/s-model_arti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
- added link robotiq_gripper_tip_frame
- added link robotiq_palm, mass 1.3; collision mesh filename=package://robotiq_s_model_visualization/meshes/s-model_arti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; visual mesh filename=package://robotiq_s_model_visualization/meshes/s-model_arti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
- link ur10_arm_ee_link: geometry collision box size=0.01 0.01 0.01; visual box size=0 0 0
Joints:
- added joint grizzly_ur10_hokuyo_joint: type fixed, parent sensor_anchor_link, child grizzly_ur10_hokuyo_link, origin xyz=1.0 0 -0.1 rpy=0 0 0, axis 0 1 0
- added joint grizzly_ur10_kinect_frame_joint: type fixed, parent sensor_anchor_link, child grizzly_ur10_kinect_frame, origin xyz=0.5 0 0.4 rpy=0 0.349065850399 0
- added joint grizzly_ur10_kinect_optical_joint: type fixed, parent grizzly_ur10_kinect_frame, child grizzly_ur10_kinect_optical_frame, origin xyz=0.0            0.0         0.0 rpy=-1.57079632679 0.0 -1.57079632679
- added joint robotiq_finger_1_joint_1: type revolute, parent robotiq_finger_1_link_0, child robotiq_finger_1_link_1, origin xyz=0.020 0 0 rpy=0 0 0, axis 0 0 1, limit lower=0 upper=3.1416 effort=100 velocity=100
- added joint robotiq_finger_1_joint_2: type revolute, parent robotiq_finger_1_link_1, child robotiq_finger_1_link_2, origin xyz=0.050 -.028 0 rpy=0 0 -0.52, axis 0 0 1, limit lower=0 upper=3.1416 effort=100 velocity=100
- added joint robotiq_finger_1_joint_3: type revolute, parent robotiq_finger_1_link_2, child robotiq_finger_1_link_3, origin xyz=0.039 0 0 rpy=0 0 0, axis 0 0 1, limit lower=0 upper=3.1416 effort=100 velocity=100
- added joint robotiq_finger_2_joint_1: type revolute, parent robotiq_finger_2_link_0, child robotiq_finger_2_link_1, origin xyz=0.020 0 0 rpy=0 0 0, axis 0 0 1, limit lower=0 upper=3.1416 effort=100 velocity=100
- added joint robotiq_finger_2_joint_2: type revolute, parent robotiq_finger_2_link_1, child robotiq_finger_2_link_2, origin xyz=0.050 -.028 0 rpy=0 0 -0.52, axis 0 0 1, limit lower=0 upper=3.1416 effort=100 velocity=100
- added joint robotiq_finger_2_joint_3: type revolute, parent robotiq_finger_2_link_2, child robotiq_finger_2_link_3, origin xyz=0.039 0 0 rpy=0 0 0, axis 0 0 1, limit lower=0 upper=3.1416 effort=100 velocity=100
- added joint robotiq_finger_middle_joint_1: type revolute, parent robotiq_finger_middle_link_0, child robotiq_finger_middle_link_1, origin xyz=0.020 0 0 rpy=0 0 0, axis 0 0 1, limit lower=0 upper=3.1416 effort=100 velocity=100
- added joint robotiq_finger_middle_joint_2: type revolute, parent robotiq_finger_middle_link_1, child robotiq_finger_middle_link_2, origin xyz=0.050 -.028 0 rpy=0 0 -0.52, axis 0 0 1, limit lower=0 upper=3.1416 effort=100 velocity=100
- added joint robotiq_finger_middle_joint_3: type revolute, parent robotiq_finger_middle_link_2, child robotiq_finger_middle_link_3, origin xyz=0.039 0 0 rpy=0 0 0, axis 0 0 1, limit lower=0 upper=3.1416 effort=100 velocity=100
- added joint robotiq_palm_finger_1_joint: type revolute, parent robotiq_palm, child robotiq_finger_1_link_0, origin xyz=-0.0455 0.0214 0.036 rpy=0 3.1416 -1.57, axis 0 1 0, limit lower=-0.16 upper=0.25 effort=100 velocity=100
- added joint robotiq_palm_finger_2_joint: type revolute, parent robotiq_palm, child robotiq_finger_2_link_0, origin xyz=-0.0455 0.0214 -0.036 rpy=0 3.1416 -1.57, axis 0 1 0, limit lower=-0.25 upper=0.16 effort=100 velocity=100
- added joint robotiq_palm_finger_middle_joint: type revolute, parent robotiq_palm, child robotiq_finger_middle_link_0, origin xyz=0.0455 0.0214 0 rpy=0 0 1.57, axis 0 0 1, limit lower=-0.25 upper=0.16 effort=100 velocity=100
- added joint ur10_arm_ee_joint: type fixed, parent robotiq_finger_middle_link_3, child robotiq_gripper_tip_frame, origin xyz=0.1 0 0 rpy=1.57 0 1.57
- added joint ur10_arm_to_gripper_joint: type fixed, parent ur10_arm_ee_link, child robotiq_palm, origin xyz=0 -0.1 0 rpy=1.57 0 1.57
- joint grizzly_ur10_joint: origin xyz=0.65 -0.21 0.03 rpy=0.0 0.0 -1.570796325 -> xyz=0.65 -0.01 0.03 rpy=0.0 0.0 -1.570796325

File: grizzly_ur10_description/urdf/ur10_arm.urdf.xacro (robot description, xacro)
@@ -26,8 +26,37 @@
 -->
 <robot xmlns:xacro="http://ros.org/wiki/xacro" name="grizzly_ur10">
-  <xacro:include filename="$(find grizzly_description)/urdf/base.urdf.xacro" />
-  <xacro:include filename="$(find grizzly_ur10_description)/urdf/ur10_arm.urdf.xacro" />
-  <xacro:include filename="$(find grizzly_ur10_description)/urdf/robotiq_gripper.urdf.xacro" />
-  <xacro:include filename="$(find grizzly_ur10_description)/urdf/grizzly_ur10_kinect.gazebo.xacro" />
-  <xacro:include filename="$(find grizzly_ur10_description)/urdf/grizzly_ur10_hokuyo.gazebo.xacro" />
+  <xacro:property name="reflect" value="-1" />
+ <xacro:include filename="$(find ur_description)/urdf/gazebo.urdf.xacro" />
+  <xacro:include filename="$(find ur_description)/urdf/ur10.urdf.xacro" />
+  <!-- Spawn arm -->
+  <xacro:ur10_robot prefix="ur10_arm_" joint_limited="true"/>
+  <!-- <xacro:ur10_robot prefix="" joint_limited="true" /> -->
+  <!-- Join arm -->
+  <joint name="grizzly_ur10_joint" type="fixed">
+    <parent link="sensor_anchor_link" />
+    <child link="ur10_arm_base_link" />
+    <origin xyz="0.65 ${reflect*0.01} 0.03" rpy="0.0 0.0 ${-pi/2}" />
+  </joint>
+  <!-- Gazebo references for self collide -->
+  <gazebo reference="ur10_arm_shoulder_link">
+      <selfCollide>true</selfCollide>
+  </gazebo>
+ <gazebo reference="ur10_arm_upper_arm_link">
+      <selfCollide>true</selfCollide>
+  </gazebo>
+ <gazebo reference="ur10_arm_forearm_link">
+      <selfCollide>true</selfCollide>
+  </gazebo>
+ <gazebo reference="ur10_arm_wrist_1_link">
+      <selfCollide>true</selfCollide>
+  </gazebo>
+ <gazebo reference="ur10_arm_wrist_3_link">
+      <selfCollide>true</selfCollide>
+  </gazebo>
+ <gazebo reference="ur10_arm_wrist_2_link">
+      <selfCollide>true</selfCollide>
+  </gazebo>
+ <gazebo reference="ur10_arm_ee_link">
+      <selfCollide>true</selfCollide>
+  </gazebo>
 </robot>

Commit message: Gripper controller loadsgit add .! but it's probably not gonna work correctly..

File: grizzly_ur10_description/urdf/grizzly_ur10.urdf (robot description, URDF)
Before this commit: robot grizzly_ur10, 35 links, 34 joints
Links:
- link robotiq_gripper_tip_frame: mass None -> 1.3; geometry visual box size=0 0 0
Joints:
- removed joint ur10_arm_ee_joint
- added joint robotiq_gripper_ee_joint: type revolute, parent robotiq_finger_middle_link_3, child robotiq_gripper_tip_frame, origin xyz=0.1 0 0 rpy=1.57 0 1.57, limit lower=-0.25 upper=0.16 effort=100 velocity=100

File: grizzly_ur10_description/urdf/robotiq_gripper.urdf.xacro (robot description, xacro)
@@ -45,5 +45,17 @@
   <!-- Chain looks like this:
    ur10_arm -> ur10_arm_ee_link -> robotiq_palm -> -->
-  <link name="robotiq_gripper_tip_frame"/>
+  <link name="robotiq_gripper_tip_frame">
+        <origin xyz="0 0 0" rpy="0 0 0" />
+	<visual>
+                    <geometry>
+                       <box size="0 0 0"/>
+                    </geometry>
+        </visual>
+	<inertial>
+		    <origin xyz="0 0 0" rpy="0 0 0"/>
+		    <mass value="1.3"/>
+		    <inertia ixx="0.006012" ixy="0.000079" ixz="-0.00024" iyy="0.012892" iyz="0" izz="0.002435" />
+	</inertial>
+  </link>
   <!-- This connects the robotiq gripper to the ur10 arm -->
   <joint name="ur10_arm_to_gripper_joint" type="fixed">
@@ -53,8 +65,9 @@
   </joint>
   <!-- this is the end effector joint before the tip frame -->
-  <joint name="robotiq_gripper_ee_joint" type="fixed">
+  <joint name="robotiq_gripper_ee_joint" type="revolute">
       <parent link="robotiq_finger_middle_link_3"/>
       <child link="robotiq_gripper_tip_frame"/>
       <origin xyz="0.1 0 0" rpy="1.57 0 1.57" />
+      <limit lower="-0.25" upper="0.16" effort="100" velocity="100"/>
   </joint>
     <!-- Gazebo macro for gripper -->

File: grizzly_ur10_description/urdf/s-model_articulated.transmission.xacro (robot description, xacro)
@@ -14,4 +14,12 @@
       <joint name="robotiq_finger_1_joint_2"/>
       <actuator name="robotiq_finger_1_joint_2_motor">
+        <hardwareInterface>EffortJointInterface</hardwareInterface>
+        <mechanicalReduction>1</mechanicalReduction>
+      </actuator>
+    </transmission>
+ <transmission name="robotiq_gripper_ee_joint_trans">
+      <type>transmission_interface/SimpleTransmission</type>
+      <joint name="robotiq_gripper_ee_joint"/>
+      <actuator name="robotiq_gripper_ee_joint_motor">
         <hardwareInterface>EffortJointInterface</hardwareInterface>
         <mechanicalReduction>1</mechanicalReduction>

Commit message: going to regenerate collision matrix

File: grizzly_ur10_description/urdf/grizzly_ur10.urdf (robot description, URDF)
Before this commit: robot grizzly_ur10, 35 links, 34 joints
Joints:
- joint robotiq_gripper_ee_joint: origin xyz=0.1 0 0 rpy=1.57 0 1.57 -> xyz=0 0 0 rpy=0 0 0
- joint ur10_arm_to_gripper_joint: origin xyz=0 -0.1 0 rpy=1.57 0 1.57 -> xyz=0.01 0 0 rpy=1.57 1.57 0
