Commit message: in the middle of robotiq gripper transition

File: grizzly_ur10_description/urdf/grizzly_ur10.urdf (robot description, URDF)
Before this commit: robot grizzly_ur10, 35 links, 34 joints
Links:
- removed link robotiq_finger_1_link_0
- removed link robotiq_finger_1_link_1
- removed link robotiq_finger_1_link_2
- removed link robotiq_finger_1_link_3
- removed link robotiq_finger_2_link_0
- removed link robotiq_finger_2_link_1
- removed link robotiq_finger_2_link_2
- removed link robotiq_finger_2_link_3
- removed link robotiq_finger_middle_link_0
- removed link robotiq_finger_middle_link_1
- removed link robotiq_finger_middle_link_2
- removed link robotiq_finger_middle_link_3
- removed link robotiq_gripper_tip_frame
- removed link robotiq_palm
- added link finger_1_link_0, mass 0.1; collision mesh filename=package://robotiq_s_model_visualization/meshes/s-model_arti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; visual mesh filename=package://robotiq_s_model_visualization/meshes/s-model_arti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
- added link finger_1_link_1, mass 0.047; collision mesh filename=package://robotiq_s_model_visualization/meshes/s-model_arti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; visual mesh filename=package://robotiq_s_model_visualization/meshes/s-model_arti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
- added link finger_1_link_2, mass 0.03284; collision mesh filename=package://robotiq_s_model_visualization/meshes/s-model_arti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; visual mesh filename=package://robotiq_s_model_visualization/meshes/s-model_arti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
- added link finger_1_link_3, mass 0.03354; collision mesh filename=package://robotiq_s_model_visualization/meshes/s-model_arti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; visual mesh filename=package://robotiq_s_model_visualization/meshes/s-model_arti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
- added link finger_1_link_median_actuating_hinge, mass 0.00359; collision box size=.02 .02 .002; visual box size=.02 .02 .002
- added link finger_1_link_median_bar, mass 0.00538; collision box size=0.0381 .0075 .002; visual box size=0.0381 .0075 .002
- added link finger_1_link_median_bar_underactuated, mass 0.00538; collision box size=0.0381 .0075 .002; visual box size=0.0381 .0075 .002
- added link finger_1_link_paradistal_hinge, mass 0.00158; collision box size=.02 0.02 .002; visual box size=.02 .02 .002
- added link finger_1_link_paramedian_hinge, mass 0.00276; collision box size=.02 .02 .002; visual box size=.02 .02 .002
- added link finger_1_link_paraproximal_actuating_hinge, mass 0.00362; collision box size=0.02286 .0075 .002; visual box size=0.02286 .0075 .002
- added link finger_1_link_paraproximal_bar, mass 0.00732; collision box size=0.05770 .0075 .002; visual box size=0.05770 .0075 .002
- added link finger_1_link_proximal_actuating_bar, mass 0.00659; collision box size=0.05398 .0075 .002; visual box size=0.05398 .0075 .002
- added link finger_1_link_proximal_actuating_hinge, mass 0.02647; collision box size=0.02858 .0075 .002; visual box size=0.02858 .0075 .002
- added link finger_2_link_0, mass 0.1; collision mesh filename=package://robotiq_s_model_visualization/meshes/s-model_arti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; visual mesh filename=package://robotiq_s_model_visualization/meshes/s-model_arti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
- added link finger_2_link_1, mass 0.047; collision mesh filename=package://robotiq_s_model_visualization/meshes/s-model_arti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; visual mesh filename=package://robotiq_s_model_visualization/meshes/s-model_arti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
- added link finger_2_link_2, mass 0.03284; collision mesh filename=package://robotiq_s_model_visualization/meshes/s-model_arti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; visual mesh filename=package://robotiq_s_model_visualization/meshes/s-model_arti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
- added link finger_2_link_3, mass 0.03354; collision mesh filename=package://robotiq_s_model_visualization/meshes/s-model_arti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; visual mesh filename=package://robotiq_s_model_visualization/meshes/s-model_arti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
- added link finger_2_link_median_actuating_hinge, mass 0.00359; collision box size=.02 .02 .002; visual box size=.02 .02 .002
- added link finger_2_link_median_bar, mass 0.00538; collision box size=0.0381 .0075 .002; visual box size=0.0381 .0075 .002
- added link finger_2_link_median_bar_underactuated, mass 0.00538; collision box size=0.0381 .0075 .002; visual box size=0.0381 .0075 .002
- added link finger_2_link_paradistal_hinge, mass 0.00158; collision box size=.02 0.02 .002; visual box size=.02 .02 .002
- added link finger_2_link_paramedian_hinge, mass 0.00276; collision box size=.02 .02 .002; visual box size=.02 .02 .002
- added link finger_2_link_paraproximal_actuating_hinge, mass 0.00362; collision box size=0.02286 .0075 .002; visual box size=0.02286 .0075 .002
- added link finger_2_link_paraproximal_bar, mass 0.00732; collision box size=0.05770 .0075 .002; visual box size=0.05770 .0075 .002
- added link finger_2_link_proximal_actuating_bar, mass 0.00659; collision box size=0.05398 .0075 .002; visual box size=0.05398 .0075 .002
- added link finger_2_link_proximal_actuating_hinge, mass 0.02647; collision box size=0.02858 .0075 .002; visual box size=0.02858 .0075 .002
- added link finger_middle_link_0, mass 0.1; collision mesh filename=package://robotiq_s_model_visualization/meshes/s-model_arti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; visual mesh filename=package://robotiq_s_model_visualization/meshes/s-model_arti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
- added link finger_middle_link_1, mass 0.047; collision mesh filename=package://robotiq_s_model_visualization/meshes/s-model_arti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; visual mesh filename=package://robotiq_s_model_visualization/meshes/s-model_arti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
- added link finger_middle_link_2, mass 0.03284; collision mesh filename=package://robotiq_s_model_visualization/meshes/s-model_arti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; visual mesh filename=package://robotiq_s_model_visualization/meshes/s-model_arti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
- added link finger_middle_link_3, mass 0.03354; collision mesh filename=package://robotiq_s_model_visualization/meshes/s-model_arti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; visual mesh filename=package://robotiq_s_model_visualization/meshes/s-model_arti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
- added link finger_middle_link_median_actuating_hinge, mass 0.00359; collision box size=.02 .02 .002; visual box size=.02 .02 .002
- added link finger_middle_link_median_bar, mass 0.00538; collision box size=0.0381 .0075 .002; visual box size=0.0381 .0075 .002
- added link finger_middle_link_median_bar_underactuated, mass 0.00538; collision box size=0.0381 .0075 .002; visual box size=0.0381 .0075 .002
- added link finger_middle_link_paradistal_hinge, mass 0.00158; collision box size=.02 0.02 .002; visual box size=.02 .02 .002
- added link finger_middle_link_paramedian_hinge, mass 0.00276; collision box size=.02 .02 .002; visual box size=.02 .02 .002
- added link finger_middle_link_paraproximal_actuating_hinge, mass 0.00362; collision box size=0.02286 .0075 .002; visual box size=0.02286 .0075 .002
- added link finger_middle_link_paraproximal_bar, mass 0.00732; collision box size=0.05770 .0075 .002; visual box size=0.05770 .0075 .002
- added link finger_middle_link_proximal_actuating_bar, mass 0.00659; collision box size=0.05398 .0075 .002; visual box size=0.05398 .0075 .002
- added link finger_middle_link_proximal_actuating_hinge, mass 0.02647; collision box size=0.02858 .0075 .002; visual box size=0.02858 .0075 .002
- added link palm, mass 1.3; collision box size=0.1 0.1 0.1; visual mesh filename=package://grizzly_ur10_description/meshes/s-model_articulat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
Joints:
- removed joint robotiq_finger_1_joint_1
- removed joint robotiq_finger_1_joint_2
- removed joint robotiq_finger_1_joint_3
- removed joint robotiq_finger_2_joint_1
- removed joint robotiq_finger_2_joint_2
- removed joint robotiq_finger_2_joint_3
- removed joint robotiq_finger_middle_joint_1
- removed joint robotiq_finger_middle_joint_2
- removed joint robotiq_finger_middle_joint_3
- removed joint robotiq_gripper_ee_joint
- removed joint robotiq_palm_finger_1_joint
- removed joint robotiq_palm_finger_2_joint
- removed joint robotiq_palm_finger_middle_joint
- removed joint ur10_arm_to_gripper_joint
- added joint finger_1_joint_1: type revolute, parent finger_1_link_0, child finger_1_link_1, origin xyz=0 0 0 rpy=0 0 -2.0906, axis 0 0 1, limit lower=0 upper=1.2217 effort=60 velocity=-1
- added joint finger_1_joint_2: type revolute, parent finger_1_link_1, child finger_1_link_2, origin xyz=0 0.05715 0 rpy=0 0 0, axis 0 0 1, limit lower=0 upper=1.5708 effort=60 velocity=-1
- added joint finger_1_joint_3: type revolute, parent finger_1_link_2, child finger_1_link_3, origin xyz=0 0.039 0 rpy=0 0 2.0906, axis 0 0 1, limit lower=-0.6632 upper=1.0471 effort=60 velocity=-1
- added joint finger_1_joint_median_actuating_hinge: type revolute, parent finger_1_link_1, child finger_1_link_median_actuating_hinge, origin xyz=0 0.05715 0.01 rpy=0 0 -0.37, axis 0 0 1, limit lower=-3.1416 upper=3.1416 effort=100 velocity=100
- added joint finger_1_joint_median_actuating_hinge_median_bar: type revolute, parent finger_1_link_median_actuating_hinge, child finger_1_link_median_bar, origin xyz=0.01625 0.01516 0 rpy=0 0 2.3215, axis 0 0 1, limit lower=-3.1416 upper=3.1416 effort=100 velocity=100
- added joint finger_1_joint_paradistal_hinge: type revolute, parent finger_1_link_2, child finger_1_link_paradistal_hinge, origin xyz=0 0.039 -0.01 rpy=0 0 0, axis 0 0 1, limit lower=-3.1416 upper=3.1416 effort=100 velocity=100
- added joint finger_1_joint_paramedian_hinge: type revolute, parent finger_1_link_1, child finger_1_link_paramedian_hinge, origin xyz=0 0.05715 -0.01 rpy=0 0 0, axis 0 0 1, limit lower=-3.1416 upper=3.1416 effort=100 velocity=100
- added joint finger_1_joint_paramedian_hinge_median_bar_underactuated: type revolute, parent finger_1_link_paramedian_hinge, child finger_1_link_median_bar_underactuated, origin xyz=0.01227 0.00329 0 rpy=0 0 1.5708, axis 0 0 1, limit lower=-3.1416 upper=3.1416 effort=100 velocity=100
- added joint finger_1_joint_paraproximal_actuating_hinge: type revolute, parent finger_1_link_0, child finger_1_link_paraproximal_actuating_hinge, origin xyz=0 0 -0.01 rpy=0 0 -2.0906, axis 0 0 1, limit lower=-3.1416 upper=3.1416 effort=100 velocity=100
- added joint finger_1_joint_paraproximal_bar: type revolute, parent finger_1_link_paraproximal_actuating_hinge, child finger_1_link_paraproximal_bar, origin xyz=0.02286 0 0 rpy=0 0 1.57, axis 0 0 1, limit lower=-3.1416 upper=3.1416 effort=100 velocity=100
- added joint finger_1_joint_proximal_actuating_bar: type revolute, parent finger_1_link_proximal_actuating_hinge, child finger_1_link_proximal_actuating_bar, origin xyz=0.02858 0 0 rpy=0 0 1.8616, axis 0 0 1, limit lower=-3.1416 upper=3.1416 effort=100 velocity=100
- added joint finger_1_joint_proximal_actuating_hinge: type revolute, parent finger_1_link_0, child finger_1_link_proximal_actuating_hinge, origin xyz=0 0 0.01 rpy=0 0 -2.0906, axis 0 0 1, limit lower=-3.1416 upper=3.1416 effort=100 velocity=100
- added joint finger_2_joint_1: type revolute, parent finger_2_link_0, child finger_2_link_1, origin xyz=0 0 0 rpy=0 0 -2.0906, axis 0 0 1, limit lower=0 upper=1.2217 effort=60 velocity=-1
- added joint finger_2_joint_2: type revolute, parent finger_2_link_1, child finger_2_link_2, origin xyz=0 0.05715 0 rpy=0 0 0, axis 0 0 1, limit lower=0 upper=1.5708 effort=60 velocity=-1
- added joint finger_2_joint_3: type revolute, parent finger_2_link_2, child finger_2_link_3, origin xyz=0 0.039 0 rpy=0 0 2.0906, axis 0 0 1, limit lower=-0.6632 upper=1.0471 effort=60 velocity=-1
- added joint finger_2_joint_median_actuating_hinge: type revolute, parent finger_2_link_1, child finger_2_link_median_actuating_hinge, origin xyz=0 0.05715 0.01 rpy=0 0 -0.37, axis 0 0 1, limit lower=-3.1416 upper=3.1416 effort=100 velocity=100
- added joint finger_2_joint_median_actuating_hinge_median_bar: type revolute, parent finger_2_link_median_actuating_hinge, child finger_2_link_median_bar, origin xyz=0.01625 0.01516 0 rpy=0 0 2.3215, axis 0 0 1, limit lower=-3.1416 upper=3.1416 effort=100 velocity=100
- added joint finger_2_joint_paradistal_hinge: type revolute, parent finger_2_link_2, child finger_2_link_paradistal_hinge, origin xyz=0 0.039 -0.01 rpy=0 0 0, axis 0 0 1, limit lower=-3.1416 upper=3.1416 effort=100 velocity=100
- added joint finger_2_joint_paramedian_hinge: type revolute, parent finger_2_link_1, child finger_2_link_paramedian_hinge, origin xyz=0 0.05715 -0.01 rpy=0 0 0, axis 0 0 1, limit lower=-3.1416 upper=3.1416 effort=100 velocity=100
- added joint finger_2_joint_paramedian_hinge_median_bar_underactuated: type revolute, parent finger_2_link_paramedian_hinge, child finger_2_link_median_bar_underactuated, origin xyz=0.01227 0.00329 0 rpy=0 0 1.5708, axis 0 0 1, limit lower=-3.1416 upper=3.1416 effort=100 velocity=100
- added joint finger_2_joint_paraproximal_actuating_hinge: type revolute, parent finger_2_link_0, child finger_2_link_paraproximal_actuating_hinge, origin xyz=0 0 -0.01 rpy=0 0 -2.0906, axis 0 0 1, limit lower=-3.1416 upper=3.1416 effort=100 velocity=100
- added joint finger_2_joint_paraproximal_bar: type revolute, parent finger_2_link_paraproximal_actuating_hinge, child finger_2_link_paraproximal_bar, origin xyz=0.02286 0 0 rpy=0 0 1.57, axis 0 0 1, limit lower=-3.1416 upper=3.1416 effort=100 velocity=100
- added joint finger_2_joint_proximal_actuating_bar: type revolute, parent finger_2_link_proximal_actuating_hinge, child finger_2_link_proximal_actuating_bar, origin xyz=0.02858 0 0 rpy=0 0 1.8616, axis 0 0 1, limit lower=-3.1416 upper=3.1416 effort=100 velocity=100
- added joint finger_2_joint_proximal_actuating_hinge: type revolute, parent finger_2_link_0, child finger_2_link_proximal_actuating_hinge, origin xyz=0 0 0.01 rpy=0 0 -2.0906, axis 0 0 1, limit lower=-3.1416 upper=3.1416 effort=100 velocity=100
- added joint finger_middle_joint_1: type revolute, parent finger_middle_link_0, child finger_middle_link_1, origin xyz=0 0 0 rpy=0 0 -2.0906, axis 0 0 1, limit lower=0 upper=1.2217 effort=60 velocity=-1
- added joint finger_middle_joint_2: type revolute, parent finger_middle_link_1, child finger_middle_link_2, origin xyz=0 0.05715 0 rpy=0 0 0, axis 0 0 1, limit lower=0 upper=1.5708 effort=60 velocity=-1
- added joint finger_middle_joint_3: type revolute, parent finger_middle_link_2, child finger_middle_link_3, origin xyz=0 0.039 0 rpy=0 0 2.0906, axis 0 0 1, limit lower=-0.6632 upper=1.0471 effort=60 velocity=-1
- added joint finger_middle_joint_median_actuating_hinge: type revolute, parent finger_middle_link_1, child finger_middle_link_median_actuating_hinge, origin xyz=0 0.05715 0.01 rpy=0 0 -0.37, axis 0 0 1, limit lower=-3.1416 upper=3.1416 effort=100 velocity=100
- added joint finger_middle_joint_median_actuating_hinge_median_bar: type revolute, parent finger_middle_link_median_actuating_hinge, child finger_middle_link_median_bar, origin xyz=0.01625 0.01516 0 rpy=0 0 2.3215, axis 0 0 1, limit lower=-3.1416 upper=3.1416 effort=100 velocity=100
- added joint finger_middle_joint_paradistal_hinge: type revolute, parent finger_middle_link_2, child finger_middle_link_paradistal_hinge, origin xyz=0 0.039 -0.01 rpy=0 0 0, axis 0 0 1, limit lower=-3.1416 upper=3.1416 effort=100 velocity=100
- added joint finger_middle_joint_paramedian_hinge: type revolute, parent finger_middle_link_1, child finger_middle_link_paramedian_hinge, origin xyz=0 0.05715 -0.01 rpy=0 0 0, axis 0 0 1, limit lower=-3.1416 upper=3.1416 effort=100 velocity=100
- added joint finger_middle_joint_paramedian_hinge_median_bar_underactuated: type revolute, parent finger_middle_link_paramedian_hinge, child finger_middle_link_median_bar_underactuated, origin xyz=0.01227 0.00329 0 rpy=0 0 1.5708, axis 0 0 1, limit lower=-3.1416 upper=3.1416 effort=100 velocity=100
- added joint finger_middle_joint_paraproximal_actuating_hinge: type revolute, parent finger_middle_link_0, child finger_middle_link_paraproximal_actuating_hinge, origin xyz=0 0 -0.01 rpy=0 0 -2.0906, axis 0 0 1, limit lower=-3.1416 upper=3.1416 effort=100 velocity=100
- added joint finger_middle_joint_paraproximal_bar: type revolute, parent finger_middle_link_paraproximal_actuating_hinge, child finger_middle_link_paraproximal_bar, origin xyz=0.02286 0 0 rpy=0 0 1.57, axis 0 0 1, limit lower=-3.1416 upper=3.1416 effort=100 velocity=100
- added joint finger_middle_joint_proximal_actuating_bar: type revolute, parent finger_middle_link_proximal_actuating_hinge, child finger_middle_link_proximal_actuating_bar, origin xyz=0.02858 0 0 rpy=0 0 1.8616, axis 0 0 1, limit lower=-3.1416 upper=3.1416 effort=100 velocity=100
- added joint finger_middle_joint_proximal_actuating_hinge: type revolute, parent finger_middle_link_0, child finger_middle_link_proximal_actuating_hinge, origin xyz=0 0 0.01 rpy=0 0 -2.0906, axis 0 0 1, limit lower=-3.1416 upper=3.1416 effort=100 velocity=100
- added joint palm_finger_1_joint: type revolute, parent palm, child finger_1_link_0, origin xyz=-0.0455 0.0214 0.036 rpy=0 3.1416 -1.57, axis 0 1 0, limit lower=-0.2967 upper=0.2967 effort=60 velocity=-1
- added joint palm_finger_2_joint: type revolute, parent palm, child finger_2_link_0, origin xyz=-0.0455 0.0214 -0.036 rpy=0 3.1416 -1.57, axis 0 1 0, limit lower=-0.2967 upper=0.2967 effort=60 velocity=-1
- added joint palm_finger_middle_joint: type revolute, parent palm, child finger_middle_link_0, origin xyz=0.0455 0.0214 0 rpy=0 0 1.57, axis 0 1 0, limit lower=0 upper=0 effort=60 velocity=-1
- added joint robotiq_hand_joint: type fixed, parent ur10_arm_ee_link, child palm, origin xyz=0 0 0 rpy=0 0 0

File: grizzly_ur10_description/urdf/robotiq_gripper.urdf.xacro (robot description, xacro)
@@ -25,15 +25,16 @@
 This program contains the description of the Grizzly + UR10 manipulator.
 -->
-<robot xmlns:xacro="http://ros.org/wiki/xacro" name="grizzly_ur10">
-  <xacro:property name="reflect" value="-1" />
+<robot xmlns:xacro="http://ros.org/wiki/xacro" name="robotiq_hand">
    <!-- Gazebo references for ur  description -->
-   <xacro:include filename="$(find ur_description)/urdf/gazebo.urdf.xacro" />
-   <xacro:include filename="$(find robotiq_s_model_visualization)/cfg/s-model_articulated_macro.xacro"/>
+   <!-- <xacro:include filename="$(find ur_description)/urdf/gazebo.urdf.xacro" />  -->
+   <!-- <xacro:include filename="$(find robotiq_s_model_visualization)/cfg/s-model_articulated_macro.xacro"/> -->
    <!-- Gazebo references -->
-   <xacro:include filename="$(find grizzly_ur10_description)/urdf/s-model_articulated.gazebo.xacro" />
+   <!-- <xacro:include filename="$(find grizzly_ur10_description)/urdf/s-model_articulated.gazebo.xacro" /> -->
    <!-- Transmission for robotiq gripper so that it can use ROS control -->
-   <xacro:include filename="$(find grizzly_ur10_description)/urdf/s-model_articulated.transmission.xacro" />
+   <!-- <xacro:include filename="$(find grizzly_ur10_description)/urdf/s-model_articulated.transmission.xacro" /> -->
+   <!-- Atlass' robotiq hand with proper underactuated joints and physics values. -->
+   <xacro:include filename="$(find grizzly_ur10_description)/urdf/robotiq_hand.urdf.xacro"/>
   <!-- Spawn gripper -->
-   <xacro:s-model_articulated prefix="robotiq_"/>
+   <!-- <xacro:s-model_articulated prefix="robotiq_"/> -->
   <!-- Note: the gripper_action_controller and MoveIt require a specific structure of the URDF so that this will work.
    end_of_robotiq_finger_tip -> joint -> tip_link -> ee_joint -> tip_frame -->
@@ -45,5 +46,5 @@
   <!-- Chain looks like this:
    ur10_arm -> ur10_arm_ee_link -> robotiq_palm -> -->
-  <link name="robotiq_gripper_tip_frame">
+ <!--  <link name="robotiq_gripper_tip_frame">
         <origin xyz="0 0 0" rpy="0 0 0" />
 	<visual>
@@ -57,21 +58,24 @@
 		    <inertia ixx="0.006012" ixy="0.000079" ixz="-0.00024" iyy="0.012892" iyz="0" izz="0.002435" />
 	</inertial>
-  </link>
+  </link> -->
   <!-- This connects the robotiq gripper to the ur10 arm -->
-  <joint name="ur10_arm_to_gripper_joint" type="fixed">
+ <!--  <joint name="ur10_arm_to_gripper_joint" type="fixed">
       <parent link="ur10_arm_ee_link"/>
       <child link="robotiq_palm"/>
       <origin xyz="0.01 0 0" rpy="1.57 1.57 0" />
-  </joint>
+  </joint>  -->
   <!-- this is the end effector joint before the tip frame -->
-  <joint name="robotiq_gripper_ee_joint" type="revolute">
+  <!-- <joint name="robotiq_gripper_ee_joint" type="revolute">
       <parent link="robotiq_finger_middle_link_3"/>
       <child link="robotiq_gripper_tip_frame"/>
       <origin xyz="0 0 0" rpy="0 0 0" />
       <limit lower="-0.25" upper="0.16" effort="100" velocity="100"/>
-  </joint>
+  </joint> -->
     <!-- Gazebo macro for gripper -->
-    <xacro:robotiq_gripper_gazebo/>
+   <!--  <xacro:robotiq_gripper_gazebo/> -->
     <!-- Instantiate transmission file -->
-    <xacro:robotiq_gripper_transmission prefix="" />
+  <!--  <xacro:robotiq_gripper_transmission prefix="" /> -->
+   <xacro:robotiq_hand prefix="" reflect="1" parent="ur10_arm_ee_link">
+      <origin xyz="0 0 0" rpy="0 0 0"/>
+   </xacro:robotiq_hand>
 </robot>
