Commit message: Added gazebo tag and working robotiq gripper in sim

File: grizzly_ur10_description/urdf/grizzly_ur10.urdf (robot description, URDF)
Before this commit: robot grizzly_ur10, 61 links, 60 joints
Links:
- removed link finger_1_link_0
- removed link finger_1_link_1
- removed link finger_1_link_2
- removed link finger_1_link_3
- removed link finger_1_link_median_actuating_hinge
- removed link finger_1_link_median_bar
- removed link finger_1_link_median_bar_underactuated
- removed link finger_1_link_paradistal_hinge
- removed link finger_1_link_paramedian_hinge
- removed link finger_1_link_paraproximal_actuating_hinge
- removed link finger_1_link_paraproximal_bar
- removed link finger_1_link_proximal_actuating_bar
- removed link finger_1_link_proximal_actuating_hinge
- removed link finger_2_link_0
- removed link finger_2_link_1
- removed link finger_2_link_2
- removed link finger_2_link_3
- removed link finger_2_link_median_actuating_hinge
- removed link finger_2_link_median_bar
- removed link finger_2_link_median_bar_underactuated
- removed link finger_2_link_paradistal_hinge
- removed link finger_2_link_paramedian_hinge
- removed link finger_2_link_paraproximal_actuating_hinge
- removed link finger_2_link_paraproximal_bar
- removed link finger_2_link_proximal_actuating_bar
- removed link finger_2_link_proximal_actuating_hinge
- removed link finger_middle_link_0
- removed link finger_middle_link_1
- removed link finger_middle_link_2
- removed link finger_middle_link_3
- removed link finger_middle_link_median_actuating_hinge
- removed link finger_middle_link_median_bar
- removed link finger_middle_link_median_bar_underactuated
- removed link finger_middle_link_paradistal_hinge
- removed link finger_middle_link_paramedian_hinge
- removed link finger_middle_link_paraproximal_actuating_hinge
- removed link finger_middle_link_paraproximal_bar
- removed link finger_middle_link_proximal_actuating_bar
- removed link finger_middle_link_proximal_actuating_hinge
- removed link palm
- added link ur10_arm_finger_1_link_0, mass 0.1; collision mesh filename=package://robotiq_s_model_visualization/meshes/s-model_arti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; visual mesh filename=package://robotiq_s_model_visualization/meshes/s-model_arti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
- added link ur10_arm_finger_1_link_1, mass 0.047; collision mesh filename=package://robotiq_s_model_visualization/meshes/s-model_arti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; visual mesh filename=package://robotiq_s_model_visualization/meshes/s-model_arti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
- added link ur10_arm_finger_1_link_2, mass 0.03284; collision mesh filename=package://robotiq_s_model_visualization/meshes/s-model_arti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; visual mesh filename=package://robotiq_s_model_visualization/meshes/s-model_arti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
- added link ur10_arm_finger_1_link_3, mass 0.03354; collision mesh filename=package://robotiq_s_model_visualization/meshes/s-model_arti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; visual mesh filename=package://robotiq_s_model_visualization/meshes/s-model_arti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
- added link ur10_arm_finger_1_link_median_actuating_hinge, mass 0.00359; collision box size=.02 .02 .002; visual box size=.02 .02 .002
- added link ur10_arm_finger_1_link_median_bar, mass 0.00538; collision box size=0.0381 .0075 .002; visual box size=0.0381 .0075 .002
- added link ur10_arm_finger_1_link_median_bar_underactuated, mass 0.00538; collision box size=0.0381 .0075 .002; visual box size=0.0381 .0075 .002
- added link ur10_arm_finger_1_link_paradistal_hinge, mass 0.00158; collision box size=.02 0.02 .002; visual box size=.02 .02 .002
- added link ur10_arm_finger_1_link_paramedian_hinge, mass 0.00276; collision box size=.02 .02 .002; visual box size=.02 .02 .002
- added link ur10_arm_finger_1_link_paraproximal_actuating_hinge, mass 0.00362; collision box size=0.02286 .0075 .002; visual box size=0.02286 .0075 .002
- added link ur10_arm_finger_1_link_paraproximal_bar, mass 0.00732; collision box size=0.05770 .0075 .002; visual box size=0.05770 .0075 .002
- added link ur10_arm_finger_1_link_proximal_actuating_bar, mass 0.00659; collision box size=0.05398 .0075 .002; visual box size=0.05398 .0075 .002
- added link ur10_arm_finger_1_link_proximal_actuating_hinge, mass 0.02647; collision box size=0.02858 .0075 .002; visual box size=0.02858 .0075 .002
- added link ur10_arm_finger_2_link_0, mass 0.1; collision mesh filename=package://robotiq_s_model_visualization/meshes/s-model_arti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; visual mesh filename=package://robotiq_s_model_visualization/meshes/s-model_arti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
- added link ur10_arm_finger_2_link_1, mass 0.047; collision mesh filename=package://robotiq_s_model_visualization/meshes/s-model_arti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; visual mesh filename=package://robotiq_s_model_visualization/meshes/s-model_arti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
- added link ur10_arm_finger_2_link_2, mass 0.03284; collision mesh filename=package://robotiq_s_model_visualization/meshes/s-model_arti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; visual mesh filename=package://robotiq_s_model_visualization/meshes/s-model_arti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
- added link ur10_arm_finger_2_link_3, mass 0.03354; collision mesh filename=package://robotiq_s_model_visualization/meshes/s-model_arti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; visual mesh filename=package://robotiq_s_model_visualization/meshes/s-model_arti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
- added link ur10_arm_finger_2_link_median_actuating_hinge, mass 0.00359; collision box size=.02 .02 .002; visual box size=.02 .02 .002
- added link ur10_arm_finger_2_link_median_bar, mass 0.00538; collision box size=0.0381 .0075 .002; visual box size=0.0381 .0075 .002
- added link ur10_arm_finger_2_link_median_bar_underactuated, mass 0.00538; collision box size=0.0381 .0075 .002; visual box size=0.0381 .0075 .002
- added link ur10_arm_finger_2_link_paradistal_hinge, mass 0.00158; collision box size=.02 0.02 .002; visual box size=.02 .02 .002
- added link ur10_arm_finger_2_link_paramedian_hinge, mass 0.00276; collision box size=.02 .02 .002; visual box size=.02 .02 .002
- added link ur10_arm_finger_2_link_paraproximal_actuating_hinge, mass 0.00362; collision box size=0.02286 .0075 .002; visual box size=0.02286 .0075 .002
- added link ur10_arm_finger_2_link_paraproximal_bar, mass 0.00732; collision box size=0.05770 .0075 .002; visual box size=0.05770 .0075 .002
- added link ur10_arm_finger_2_link_proximal_actuating_bar, mass 0.00659; collision box size=0.05398 .0075 .002; visual box size=0.05398 .0075 .002
- added link ur10_arm_finger_2_link_proximal_actuating_hinge, mass 0.02647; collision box size=0.02858 .0075 .002; visual box size=0.02858 .0075 .002
- added link ur10_arm_finger_middle_link_0, mass 0.1; collision mesh filename=package://robotiq_s_model_visualization/meshes/s-model_arti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; visual mesh filename=package://robotiq_s_model_visualization/meshes/s-model_arti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
- added link ur10_arm_finger_middle_link_1, mass 0.047; collision mesh filename=package://robotiq_s_model_visualization/meshes/s-model_arti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; visual mesh filename=package://robotiq_s_model_visualization/meshes/s-model_arti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
- added link ur10_arm_finger_middle_link_2, mass 0.03284; collision mesh filename=package://robotiq_s_model_visualization/meshes/s-model_arti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; visual mesh filename=package://robotiq_s_model_visualization/meshes/s-model_arti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
- added link ur10_arm_finger_middle_link_3, mass 0.03354; collision mesh filename=package://robotiq_s_model_visualization/meshes/s-model_arti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; visual mesh filename=package://robotiq_s_model_visualization/meshes/s-model_arti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
- added link ur10_arm_finger_middle_link_median_actuating_hinge, mass 0.00359; collision box size=.02 .02 .002; visual box size=.02 .02 .002
- added link ur10_arm_finger_middle_link_median_bar, mass 0.00538; collision box size=0.0381 .0075 .002; visual box size=0.0381 .0075 .002
- added link ur10_arm_finger_middle_link_median_bar_underactuated, mass 0.00538; collision box size=0.0381 .0075 .002; visual box size=0.0381 .0075 .002
- added link ur10_arm_finger_middle_link_paradistal_hinge, mass 0.00158; collision box size=.02 0.02 .002; visual box size=.02 .02 .002
- added link ur10_arm_finger_middle_link_paramedian_hinge, mass 0.00276; collision box size=.02 .02 .002; visual box size=.02 .02 .002
- added link ur10_arm_finger_middle_link_paraproximal_actuating_hinge, mass 0.00362; collision box size=0.02286 .0075 .002; visual box size=0.02286 .0075 .002
- added link ur10_arm_finger_middle_link_paraproximal_bar, mass 0.00732; collision box size=0.05770 .0075 .002; visual box size=0.05770 .0075 .002
- added link ur10_arm_finger_middle_link_proximal_actuating_bar, mass 0.00659; collision box size=0.05398 .0075 .002; visual box size=0.05398 .0075 .002
- added link ur10_arm_finger_middle_link_proximal_actuating_hinge, mass 0.02647; collision box size=0.02858 .0075 .002; visual box size=0.02858 .0075 .002
- added link ur10_arm_palm, mass 1.3; collision box size=0.1 0.1 0.1; visual mesh filename=package://grizzly_ur10_description/meshes/s-model_articulat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
Joints:
- removed joint finger_1_joint_1
- removed joint finger_1_joint_2
- removed joint finger_1_joint_3
- removed joint finger_1_joint_median_actuating_hinge
- removed joint finger_1_joint_median_actuating_hinge_median_bar
- removed joint finger_1_joint_paradistal_hinge
- removed joint finger_1_joint_paramedian_hinge
- removed joint finger_1_joint_paramedian_hinge_median_bar_underactuated
- removed joint finger_1_joint_paraproximal_actuating_hinge
- removed joint finger_1_joint_paraproximal_bar
- removed joint finger_1_joint_proximal_actuating_bar
- removed joint finger_1_joint_proximal_actuating_hinge
- removed joint finger_2_joint_1
- removed joint finger_2_joint_2
- removed joint finger_2_joint_3
- removed joint finger_2_joint_median_actuating_hinge
- removed joint finger_2_joint_median_actuating_hinge_median_bar
- removed joint finger_2_joint_paradistal_hinge
- removed joint finger_2_joint_paramedian_hinge
- removed joint finger_2_joint_paramedian_hinge_median_bar_underactuated
- removed joint finger_2_joint_paraproximal_actuating_hinge
- removed joint finger_2_joint_paraproximal_bar
- removed joint finger_2_joint_proximal_actuating_bar
- removed joint finger_2_joint_proximal_actuating_hinge
- removed joint finger_middle_joint_1
- removed joint finger_middle_joint_2
- removed joint finger_middle_joint_3
- removed joint finger_middle_joint_median_actuating_hinge
- removed joint finger_middle_joint_median_actuating_hinge_median_bar
- removed joint finger_middle_joint_paradistal_hinge
- removed joint finger_middle_joint_paramedian_hinge
- removed joint finger_middle_joint_paramedian_hinge_median_bar_underactuated
- removed joint finger_middle_joint_paraproximal_actuating_hinge
- removed joint finger_middle_joint_paraproximal_bar
- removed joint finger_middle_joint_proximal_actuating_bar
- removed joint finger_middle_joint_proximal_actuating_hinge
- removed joint palm_finger_1_joint
- removed joint palm_finger_2_joint
- removed joint palm_finger_middle_joint
- removed joint robotiq_hand_joint
- added joint ur10_arm_finger_1_joint_1: type revolute, parent ur10_arm_finger_1_link_0, child ur10_arm_finger_1_link_1, origin xyz=0 0 0 rpy=0 0 -2.0906, axis 0 0 1, limit lower=0 upper=1.2217 effort=60 velocity=-1
- added joint ur10_arm_finger_1_joint_2: type revolute, parent ur10_arm_finger_1_link_1, child ur10_arm_finger_1_link_2, origin xyz=0 0.05715 0 rpy=0 0 0, axis 0 0 1, limit lower=0 upper=1.5708 effort=60 velocity=-1
- added joint ur10_arm_finger_1_joint_3: type revolute, parent ur10_arm_finger_1_link_2, child ur10_arm_finger_1_link_3, origin xyz=0 0.039 0 rpy=0 0 2.0906, axis 0 0 1, limit lower=-0.6632 upper=1.0471 effort=60 velocity=-1
- added joint ur10_arm_finger_1_joint_median_actuating_hinge: type revolute, parent ur10_arm_finger_1_link_1, child ur10_arm_finger_1_link_median_actuating_hinge, origin xyz=0 0.05715 0.01 rpy=0 0 -0.37, axis 0 0 1, limit lower=-3.1416 upper=3.1416 effort=100 velocity=100
- added joint ur10_arm_finger_1_joint_median_actuating_hinge_median_bar: type revolute, parent ur10_arm_finger_1_link_median_actuating_hinge, child ur10_arm_finger_1_link_median_bar, origin xyz=0.01625 0.01516 0 rpy=0 0 2.3215, axis 0 0 1, limit lower=-3.1416 upper=3.1416 effort=100 velocity=100
- added joint ur10_arm_finger_1_joint_paradistal_hinge: type revolute, parent ur10_arm_finger_1_link_2, child ur10_arm_finger_1_link_paradistal_hinge, origin xyz=0 0.039 -0.01 rpy=0 0 0, axis 0 0 1, limit lower=-3.1416 upper=3.1416 effort=100 velocity=100
- added joint ur10_arm_finger_1_joint_paramedian_hinge: type revolute, parent ur10_arm_finger_1_link_1, child ur10_arm_finger_1_link_paramedian_hinge, origin xyz=0 0.05715 -0.01 rpy=0 0 0, axis 0 0 1, limit lower=-3.1416 upper=3.1416 effort=100 velocity=100
- added joint ur10_arm_finger_1_joint_paramedian_hinge_median_bar_underactuated: type revolute, parent ur10_arm_finger_1_link_paramedian_hinge, child ur10_arm_finger_1_link_median_bar_underactuated, origin xyz=0.01227 0.00329 0 rpy=0 0 1.5708, axis 0 0 1, limit lower=-3.1416 upper=3.1416 effort=100 velocity=100
- added joint ur10_arm_finger_1_joint_paraproximal_actuating_hinge: type revolute, parent ur10_arm_finger_1_link_0, child ur10_arm_finger_1_link_paraproximal_actuating_hinge, origin xyz=0 0 -0.01 rpy=0 0 -2.0906, axis 0 0 1, limit lower=-3.1416 upper=3.1416 effort=100 velocity=100
- added joint ur10_arm_finger_1_joint_paraproximal_bar: type revolute, parent ur10_arm_finger_1_link_paraproximal_actuating_hinge, child ur10_arm_finger_1_link_paraproximal_bar, origin xyz=0.02286 0 0 rpy=0 0 1.57, axis 0 0 1, limit lower=-3.1416 upper=3.1416 effort=100 velocity=100
- added joint ur10_arm_finger_1_joint_proximal_actuating_bar: type revolute, parent ur10_arm_finger_1_link_proximal_actuating_hinge, child ur10_arm_finger_1_link_proximal_actuating_bar, origin xyz=0.02858 0 0 rpy=0 0 1.8616, axis 0 0 1, limit lower=-3.1416 upper=3.1416 effort=100 velocity=100
- added joint ur10_arm_finger_1_joint_proximal_actuating_hinge: type revolute, parent ur10_arm_finger_1_link_0, child ur10_arm_finger_1_link_proximal_actuating_hinge, origin xyz=0 0 0.01 rpy=0 0 -2.0906, axis 0 0 1, limit lower=-3.1416 upper=3.1416 effort=100 velocity=100
- added joint ur10_arm_finger_2_joint_1: type revolute, parent ur10_arm_finger_2_link_0, child ur10_arm_finger_2_link_1, origin xyz=0 0 0 rpy=0 0 -2.0906, axis 0 0 1, limit lower=0 upper=1.2217 effort=60 velocity=-1
- added joint ur10_arm_finger_2_joint_2: type revolute, parent ur10_arm_finger_2_link_1, child ur10_arm_finger_2_link_2, origin xyz=0 0.05715 0 rpy=0 0 0, axis 0 0 1, limit lower=0 upper=1.5708 effort=60 velocity=-1
- added joint ur10_arm_finger_2_joint_3: type revolute, parent ur10_arm_finger_2_link_2, child ur10_arm_finger_2_link_3, origin xyz=0 0.039 0 rpy=0 0 2.0906, axis 0 0 1, limit lower=-0.6632 upper=1.0471 effort=60 velocity=-1
- added joint ur10_arm_finger_2_joint_median_actuating_hinge: type revolute, parent ur10_arm_finger_2_link_1, child ur10_arm_finger_2_link_median_actuating_hinge, origin xyz=0 0.05715 0.01 rpy=0 0 -0.37, axis 0 0 1, limit lower=-3.1416 upper=3.1416 effort=100 velocity=100
- added joint ur10_arm_finger_2_joint_median_actuating_hinge_median_bar: type revolute, parent ur10_arm_finger_2_link_median_actuating_hinge, child ur10_arm_finger_2_link_median_bar, origin xyz=0.01625 0.01516 0 rpy=0 0 2.3215, axis 0 0 1, limit lower=-3.1416 upper=3.1416 effort=100 velocity=100
- added joint ur10_arm_finger_2_joint_paradistal_hinge: type revolute, parent ur10_arm_finger_2_link_2, child ur10_arm_finger_2_link_paradistal_hinge, origin xyz=0 0.039 -0.01 rpy=0 0 0, axis 0 0 1, limit lower=-3.1416 upper=3.1416 effort=100 velocity=100
- added joint ur10_arm_finger_2_joint_paramedian_hinge: type revolute, parent ur10_arm_finger_2_link_1, child ur10_arm_finger_2_link_paramedian_hinge, origin xyz=0 0.05715 -0.01 rpy=0 0 0, axis 0 0 1, limit lower=-3.1416 upper=3.1416 effort=100 velocity=100
- added joint ur10_arm_finger_2_joint_paramedian_hinge_median_bar_underactuated: type revolute, parent ur10_arm_finger_2_link_paramedian_hinge, child ur10_arm_finger_2_link_median_bar_underactuated, origin xyz=0.01227 0.00329 0 rpy=0 0 1.5708, axis 0 0 1, limit lower=-3.1416 upper=3.1416 effort=100 velocity=100
- added joint ur10_arm_finger_2_joint_paraproximal_actuating_hinge: type revolute, parent ur10_arm_finger_2_link_0, child ur10_arm_finger_2_link_paraproximal_actuating_hinge, origin xyz=0 0 -0.01 rpy=0 0 -2.0906, axis 0 0 1, limit lower=-3.1416 upper=3.1416 effort=100 velocity=100
- added joint ur10_arm_finger_2_joint_paraproximal_bar: type revolute, parent ur10_arm_finger_2_link_paraproximal_actuating_hinge, child ur10_arm_finger_2_link_paraproximal_bar, origin xyz=0.02286 0 0 rpy=0 0 1.57, axis 0 0 1, limit lower=-3.1416 upper=3.1416 effort=100 velocity=100
- added joint ur10_arm_finger_2_joint_proximal_actuating_bar: type revolute, parent ur10_arm_finger_2_link_proximal_actuating_hinge, child ur10_arm_finger_2_link_proximal_actuating_bar, origin xyz=0.02858 0 0 rpy=0 0 1.8616, axis 0 0 1, limit lower=-3.1416 upper=3.1416 effort=100 velocity=100
- added joint ur10_arm_finger_2_joint_proximal_actuating_hinge: type revolute, parent ur10_arm_finger_2_link_0, child ur10_arm_finger_2_link_proximal_actuating_hinge, origin xyz=0 0 0.01 rpy=0 0 -2.0906, axis 0 0 1, limit lower=-3.1416 upper=3.1416 effort=100 velocity=100
- added joint ur10_arm_finger_middle_joint_1: type revolute, parent ur10_arm_finger_middle_link_0, child ur10_arm_finger_middle_link_1, origin xyz=0 0 0 rpy=0 0 -2.0906, axis 0 0 1, limit lower=0 upper=1.2217 effort=60 velocity=-1
- added joint ur10_arm_finger_middle_joint_2: type revolute, parent ur10_arm_finger_middle_link_1, child ur10_arm_finger_middle_link_2, origin xyz=0 0.05715 0 rpy=0 0 0, axis 0 0 1, limit lower=0 upper=1.5708 effort=60 velocity=-1
- added joint ur10_arm_finger_middle_joint_3: type revolute, parent ur10_arm_finger_middle_link_2, child ur10_arm_finger_middle_link_3, origin xyz=0 0.039 0 rpy=0 0 2.0906, axis 0 0 1, limit lower=-0.6632 upper=1.0471 effort=60 velocity=-1
- added joint ur10_arm_finger_middle_joint_median_actuating_hinge: type revolute, parent ur10_arm_finger_middle_link_1, child ur10_arm_finger_middle_link_median_actuating_hinge, origin xyz=0 0.05715 0.01 rpy=0 0 -0.37, axis 0 0 1, limit lower=-3.1416 upper=3.1416 effort=100 velocity=100
- added joint ur10_arm_finger_middle_joint_median_actuating_hinge_median_bar: type revolute, parent ur10_arm_finger_middle_link_median_actuating_hinge, child ur10_arm_finger_middle_link_median_bar, origin xyz=0.01625 0.01516 0 rpy=0 0 2.3215, axis 0 0 1, limit lower=-3.1416 upper=3.1416 effort=100 velocity=100
- added joint ur10_arm_finger_middle_joint_paradistal_hinge: type revolute, parent ur10_arm_finger_middle_link_2, child ur10_arm_finger_middle_link_paradistal_hinge, origin xyz=0 0.039 -0.01 rpy=0 0 0, axis 0 0 1, limit lower=-3.1416 upper=3.1416 effort=100 velocity=100
- added joint ur10_arm_finger_middle_joint_paramedian_hinge: type revolute, parent ur10_arm_finger_middle_link_1, child ur10_arm_finger_middle_link_paramedian_hinge, origin xyz=0 0.05715 -0.01 rpy=0 0 0, axis 0 0 1, limit lower=-3.1416 upper=3.1416 effort=100 velocity=100
- added joint ur10_arm_finger_middle_joint_paramedian_hinge_median_bar_underactuated: type revolute, parent ur10_arm_finger_middle_link_paramedian_hinge, child ur10_arm_finger_middle_link_median_bar_underactuated, origin xyz=0.01227 0.00329 0 rpy=0 0 1.5708, axis 0 0 1, limit lower=-3.1416 upper=3.1416 effort=100 velocity=100
- added joint ur10_arm_finger_middle_joint_paraproximal_actuating_hinge: type revolute, parent ur10_arm_finger_middle_link_0, child ur10_arm_finger_middle_link_paraproximal_actuating_hinge, origin xyz=0 0 -0.01 rpy=0 0 -2.0906, axis 0 0 1, limit lower=-3.1416 upper=3.1416 effort=100 velocity=100
- added joint ur10_arm_finger_middle_joint_paraproximal_bar: type revolute, parent ur10_arm_finger_middle_link_paraproximal_actuating_hinge, child ur10_arm_finger_middle_link_paraproximal_bar, origin xyz=0.02286 0 0 rpy=0 0 1.57, axis 0 0 1, limit lower=-3.1416 upper=3.1416 effort=100 velocity=100
- added joint ur10_arm_finger_middle_joint_proximal_actuating_bar: type revolute, parent ur10_arm_finger_middle_link_proximal_actuating_hinge, child ur10_arm_finger_middle_link_proximal_actuating_bar, origin xyz=0.02858 0 0 rpy=0 0 1.8616, axis 0 0 1, limit lower=-3.1416 upper=3.1416 effort=100 velocity=100
- added joint ur10_arm_finger_middle_joint_proximal_actuating_hinge: type revolute, parent ur10_arm_finger_middle_link_0, child ur10_arm_finger_middle_link_proximal_actuating_hinge, origin xyz=0 0 0.01 rpy=0 0 -2.0906, axis 0 0 1, limit lower=-3.1416 upper=3.1416 effort=100 velocity=100
- added joint ur10_arm_palm_finger_1_joint: type revolute, parent ur10_arm_palm, child ur10_arm_finger_1_link_0, origin xyz=-0.0455 0.0214 0.036 rpy=0 3.1416 -1.57, axis 0 1 0, limit lower=-0.2967 upper=0.2967 effort=60 velocity=-1
- added joint ur10_arm_palm_finger_2_joint: type revolute, parent ur10_arm_palm, child ur10_arm_finger_2_link_0, origin xyz=-0.0455 0.0214 -0.036 rpy=0 3.1416 -1.57, axis 0 1 0, limit lower=-0.2967 upper=0.2967 effort=60 velocity=-1
- added joint ur10_arm_palm_finger_middle_joint: type revolute, parent ur10_arm_palm, child ur10_arm_finger_middle_link_0, origin xyz=0.0455 0.0214 0 rpy=0 0 1.57, axis 0 1 0, limit lower=0 upper=0 effort=60 velocity=-1
- added joint ur10_arm_robotiq_hand_joint: type fixed, parent ur10_arm_ee_link, child ur10_arm_palm, origin xyz=0 0 0 rpy=0 0 0

File: grizzly_ur10_description/urdf/robotiq_gripper.urdf.xacro (robot description, xacro)
@@ -73,15 +73,16 @@
   </joint> -->
     <!-- Gazebo macro for gripper -->
-   <!--  <xacro:robotiq_gripper_gazebo/> -->
+     <!-- <xacro:robotiq_gripper_gazebo/> -->
     <!-- Instantiate transmission file -->
   <!--  <xacro:robotiq_gripper_transmission prefix="" /> -->
-  <!--  <xacro:robotiq_hand prefix="ur10_arm_" reflect="1" parent="ur10_arm_ee_link">
+   <xacro:robotiq_hand prefix="ur10_arm_" reflect="1" parent="ur10_arm_ee_link">
       <origin xyz="0 0 0" rpy="0 0 0"/>
-   </xacro:robotiq_hand> -->
-   <!-- <gazebo>
-    <plugin name="left_robotiq_hand_plugin" filename="libRobotiqHandPlugin.so">
-      <side>left</side>
-      <kp_position>5.0</kp_position>
-      <kd_position>0.5</kd_position>
-    </plugin> -->
+   </xacro:robotiq_hand>
+    <gazebo>
+	    <plugin name="robotiq_hand_plugin" filename="libRobotiqHandPlugin.so">
+	      <side>left</side>
+	      <kp_position>5.0</kp_position>
+	      <kd_position>0.5</kd_position>
+	     </plugin>
+     </gazebo>
 </robot>
