Commit message: Added robotiq gripper to model

File: grizzly_ur10_description/urdf/base_with_manipulator.urdf.xacro (robot description, xacro)
@@ -28,4 +28,4 @@
   <xacro:include filename="$(find grizzly_description)/urdf/base.urdf.xacro" />
   <xacro:include filename="$(find grizzly_ur10_description)/urdf/ur10_arm.urdf.xacro" />
-  <xacro:include filename="$(find grizzly_ur10_description/urdf/robotiq_gripper.urdf.xacro" />
+  <xacro:include filename="$(find grizzly_ur10_description)/urdf/robotiq_gripper.urdf.xacro" />
 </robot>

File: grizzly_ur10_description/urdf/grizzly_ur10.urdf (robot description, URDF)
Before this commit: robot grizzly_ur10, 18 links, 17 joints
Links:
- added link robotiq_finger_1_link_0, mass 0.05; collision mesh filename=package://robotiq_s_model_visualization/meshes/s-model_arti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; visual mesh filename=package://robotiq_s_model_visualization/meshes/s-model_arti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
- added link robotiq_finger_1_link_1, mass 0.15; collision mesh filename=package://robotiq_s_model_visualization/meshes/s-model_arti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; visual mesh filename=package://robotiq_s_model_visualization/meshes/s-model_arti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
- added link robotiq_finger_1_link_2, mass 0.15; collision mesh filename=package://robotiq_s_model_visualization/meshes/s-model_arti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; visual mesh filename=package://robotiq_s_model_visualization/meshes/s-model_arti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
- added link robotiq_finger_1_link_3, mass 0.05; collision mesh filename=package://robotiq_s_model_visualization/meshes/s-model_arti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; visual mesh filename=package://robotiq_s_model_visualization/meshes/s-model_arti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
- added link robotiq_finger_2_link_0, mass 0.05; collision mesh filename=package://robotiq_s_model_visualization/meshes/s-model_arti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; visual mesh filename=package://robotiq_s_model_visualization/meshes/s-model_arti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
- added link robotiq_finger_2_link_1, mass 0.15; collision mesh filename=package://robotiq_s_model_visualization/meshes/s-model_arti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; visual mesh filename=package://robotiq_s_model_visualization/meshes/s-model_arti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
- added link robotiq_finger_2_link_2, mass 0.15; collision mesh filename=package://robotiq_s_model_visualization/meshes/s-model_arti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; visual mesh filename=package://robotiq_s_model_visualization/meshes/s-model_arti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
- added link robotiq_finger_2_link_3, mass 0.05; collision mesh filename=package://robotiq_s_model_visualization/meshes/s-model_arti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; visual mesh filename=package://robotiq_s_model_visualization/meshes/s-model_arti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
- added link robotiq_finger_middle_link_0, mass 0.05; collision mesh filename=package://robotiq_s_model_visualization/meshes/s-model_arti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; visual mesh filename=package://robotiq_s_model_visualization/meshes/s-model_arti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
- added link robotiq_finger_middle_link_1, mass 0.15; collision mesh filename=package://robotiq_s_model_visualization/meshes/s-model_arti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; visual mesh filename=package://robotiq_s_model_visualization/meshes/s-model_arti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
- added link robotiq_finger_middle_link_2, mass 0.15; collision mesh filename=package://robotiq_s_model_visualization/meshes/s-model_arti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; visual mesh filename=package://robotiq_s_model_visualization/meshes/s-model_arti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
- added link robotiq_finger_middle_link_3, mass 0.05; collision mesh filename=package://robotiq_s_model_visualization/meshes/s-model_arti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; visual mesh filename=package://robotiq_s_model_visualization/meshes/s-model_arti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
- added link robotiq_palm; collision mesh filename=package://robotiq_s_model_visualization/meshes/s-model_arti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; visual mesh filename=package://robotiq_s_model_visualization/meshes/s-model_arti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
Joints:
- added joint ee_joint: type fixed, parent ur10_arm_ee_link, child robotiq_palm, origin xyz=0 0 0 rpy=1.57 0.78 0.78
- added joint robotiq_finger_1_joint_1: type revolute, parent robotiq_finger_1_link_0, child robotiq_finger_1_link_1, origin xyz=0.020 0 0 rpy=0 0 0, axis 0 0 1, limit lower=0 upper=3.1416 effort=100 velocity=100
- added joint robotiq_finger_1_joint_2: type revolute, parent robotiq_finger_1_link_1, child robotiq_finger_1_link_2, origin xyz=0.050 -.028 0 rpy=0 0 -0.52, axis 0 0 1, limit lower=0 upper=3.1416 effort=100 velocity=100
- added joint robotiq_finger_1_joint_3: type revolute, parent robotiq_finger_1_link_2, child robotiq_finger_1_link_3, origin xyz=0.039 0 0 rpy=0 0 0, axis 0 0 1, limit lower=0 upper=3.1416 effort=100 velocity=100
- added joint robotiq_finger_2_joint_1: type revolute, parent robotiq_finger_2_link_0, child robotiq_finger_2_link_1, origin xyz=0.020 0 0 rpy=0 0 0, axis 0 0 1, limit lower=0 upper=3.1416 effort=100 velocity=100
- added joint robotiq_finger_2_joint_2: type revolute, parent robotiq_finger_2_link_1, child robotiq_finger_2_link_2, origin xyz=0.050 -.028 0 rpy=0 0 -0.52, axis 0 0 1, limit lower=0 upper=3.1416 effort=100 velocity=100
- added joint robotiq_finger_2_joint_3: type revolute, parent robotiq_finger_2_link_2, child robotiq_finger_2_link_3, origin xyz=0.039 0 0 rpy=0 0 0, axis 0 0 1, limit lower=0 upper=3.1416 effort=100 velocity=100
- added joint robotiq_finger_middle_joint_1: type revolute, parent robotiq_finger_middle_link_0, child robotiq_finger_middle_link_1, origin xyz=0.020 0 0 rpy=0 0 0, axis 0 0 1, limit lower=0 upper=3.1416 effort=100 velocity=100
- added joint robotiq_finger_middle_joint_2: type revolute, parent robotiq_finger_middle_link_1, child robotiq_finger_middle_link_2, origin xyz=0.050 -.028 0 rpy=0 0 -0.52, axis 0 0 1, limit lower=0 upper=3.1416 effort=100 velocity=100
- added joint robotiq_finger_middle_joint_3: type revolute, parent robotiq_finger_middle_link_2, child robotiq_finger_middle_link_3, origin xyz=0.039 0 0 rpy=0 0 0, axis 0 0 1, limit lower=0 upper=3.1416 effort=100 velocity=100
- added joint robotiq_palm_finger_1_joint: type revolute, parent robotiq_palm, child robotiq_finger_1_link_0, origin xyz=-0.0455 0.0214 0.036 rpy=0 3.1416 -1.57, axis 0 1 0, limit lower=-0.16 upper=0.25 effort=100 velocity=100
- added joint robotiq_palm_finger_2_joint: type revolute, parent robotiq_palm, child robotiq_finger_2_link_0, origin xyz=-0.0455 0.0214 -0.036 rpy=0 3.1416 -1.57, axis 0 1 0, limit lower=-0.25 upper=0.16 effort=100 velocity=100
- added joint robotiq_palm_finger_middle_joint: type fixed, parent robotiq_palm, child robotiq_finger_middle_link_0, origin xyz=0.0455 0.0214 0 rpy=0 0 1.57, axis 0 0 1

File: grizzly_ur10_description/urdf/robotiq_gripper.urdf.xacro (robot description, xacro)
@@ -28,13 +28,12 @@
   <xacro:property name="reflect" value="-1" />
  <xacro:include filename="$(find ur_description)/urdf/gazebo.urdf.xacro" />
-  <xacro:include filename="$(find ur_description)/urdf/ur10_arm.urdf.xacro" />
-  <xacro:include filename="$(find robotiq_s_model_visualization)/cfg/s-model_articulated_macro.urdf.xacro" />
+  <xacro:include filename="$(find robotiq_s_model_visualization)/cfg/s-model_articulated_macro.xacro" />
   <!-- Spawn gripper -->
   <xacro:s-model_articulated prefix="robotiq_"/>
   <!-- Add robotiq gripper -->
   <joint name="ee_joint" type="fixed">
-      <parent link="ee_link"/>
+      <parent link="ur10_arm_ee_link"/>
       <child link="robotiq_palm"/>
-      <origin xyz="0 0 0" rpy="0 0 0" />
+      <origin xyz="0 0 0" rpy="3.14 0 1.57" />
   </joint>
 </robot>

Commit message: Added more frames for kinect sensor

File: grizzly_ur10_description/urdf/base_with_manipulator.urdf.xacro (robot description, xacro)
@@ -29,3 +29,4 @@
   <xacro:include filename="$(find grizzly_ur10_description)/urdf/ur10_arm.urdf.xacro" />
   <xacro:include filename="$(find grizzly_ur10_description)/urdf/robotiq_gripper.urdf.xacro" />
+  <xacro:include filename="$(find grizzly_ur10_description)/urdf/grizzly_ur10_kinect.gazebo.xacro" />
 </robot>

File: grizzly_ur10_description/urdf/grizzly_ur10.urdf (robot description, URDF)
Before this commit: robot grizzly_ur10, 32 links, 31 joints
Links:
- added link grizzly_ur10_kinect_frame
Joints:
- added joint grizzly_ur10_kinect_frame_joint: type None, parent sensor_anchor_link, child grizzly_ur10_kinect_frame, origin xyz=0 0 0 rpy=0 0 0
- joint grizzly_ur10_joint: origin xyz=0.65 -0.21 0.03 rpy=0.0 0.0 -1.570796325 -> xyz=0.65 -0.01 0.03 rpy=0.0 0.0 -1.570796325

Commit message: Working properly; sensors in correct positions; planning

File: grizzly_ur10_description/urdf/base_with_manipulator.urdf.xacro (robot description, xacro)
@@ -30,3 +30,4 @@
   <xacro:include filename="$(find grizzly_ur10_description)/urdf/robotiq_gripper.urdf.xacro" />
   <xacro:include filename="$(find grizzly_ur10_description)/urdf/grizzly_ur10_kinect.gazebo.xacro" />
+  <xacro:include filename="$(find grizzly_ur10_description)/urdf/grizzly_ur10_hokuyo.gazebo.xacro" />
 </robot>

File: grizzly_ur10_description/urdf/grizzly_ur10_kinect.gazebo.xacro (robot description, xacro)
@@ -2,49 +2,9 @@
 <robot xmlns:xacro="http://ros.org/wiki/xacro" name="grizzly_ur10_kinect">
   <xacro:property name="reflect" value="-1" />
-<xacro:include filename="$(find pr2_description)/urdf/sensors/kinect_camera.gazebo.xacro"/>
-<!-- Add the kinect frame to the grizzly_ur10 -->
-<link name="grizzly_ur10_kinect_frame"/>
-<link name="grizzly_ur10_kinect_optical_frame"/>
-<!-- Kinect frame addition -->
-<joint name="grizzly_ur10_kinect_frame_joint" type="fixed">
-    <parent link="grizzly_ur10_kinect_link"/>
-    <child link="grizzly_ur10_kinect_frame"/>
-    <origin xyz="0 0 0" rpy="0 0 0"/>
-</joint>
-<!-- Optical frame addition -->
-<joint name="grizzly_ur10_kinect_optical_frame_joint" type="fixed">
-    <parent link="grizzly_ur10_kinect_frame"/>
-    <child link="grizzly_ur10_kinect_optical_frame"/>
-    <origin xyz="0 0 0" rpy="0 0 -${M_PI/2}"/>
-</joint>
-<!-- Adding the actual kinect model -->
-<link name="grizzly_ur10_kinect_link">
-	<visual>
-		<origin xyz="0 0 0" rpy="-${M_PI/2} 0 ${M_PI}"/>
-		<geometry>
-		<mesh filename="package://grizzly_ur10_description/meshes/sensors/kinect.dae"/>
-		</geometry>
-	</visual>
-	<collision>
-		<origin xyz="0.0 0.0 0.0" rpy="0 0 0"/>
-		<geometry>
-		<box size="0.07271 0.27794 0.073"/>
-		</geometry>
-	</collision>
-	<inertial>
-		<mass value="0.001" />
-		<origin xyz="0 0 0" />
-		<inertia ixx="0.0001" ixy="0.0" ixz="0.0"
-		iyy="0.0001" iyz="0.0"
-		izz="0.0001" />
-	</inertial>
-</link>
-<!-- Connect kinect to robot -->
-<joint name="grizzly_ur10_kinect_joint" type="fixed">
-    <parent link="sensor_anchor_link"/>
-    <child link="grizzly_ur10_kinect_link"/>
-    <origin xyz="0.9 0 0" rpy="${M_PI/2} ${M_PI} ${M_PI/2}"/>
-</joint>
-<!-- Add the kinect to the grizzly_ur10 project. This macro looks for ${name}_frame as its target frame. -->
-<xacro:kinect_camera_gazebo_v0 name="grizzly_ur10_kinect"/>
+<xacro:include filename="$(find pr2_description)/urdf/sensors/kinect_camera.urdf.xacro"/>
+<xacro:include filename="$(find pr2_description)/urdf/common.xacro"/>
+<!-- Add kinect -->
+<xacro:kinect_camera_v0 name="grizzly_ur10_kinect" parent="sensor_anchor_link">
+    <origin xyz="0.9 0 0" rpy="0 0 0"/>
+</xacro:kinect_camera_v0>
 </robot>

Commit message: Added more collision disables

File: grizzly_ur10_description/urdf/base_with_manipulator.urdf.xacro (robot description, xacro)
@@ -29,5 +29,5 @@
   <xacro:include filename="$(find grizzly_ur10_description)/urdf/ur10_arm.urdf.xacro" />
   <xacro:include filename="$(find grizzly_ur10_description)/urdf/robotiq_gripper.urdf.xacro" />
-  <xacro:include filename="$(find grizzly_ur10_description)/urdf/grizzly_ur10_kinect.gazebo.xacro" />
+<!--  <xacro:include filename="$(find grizzly_ur10_description)/urdf/grizzly_ur10_kinect.gazebo.xacro" /> -->
   <xacro:include filename="$(find grizzly_ur10_description)/urdf/grizzly_ur10_hokuyo.gazebo.xacro" />
 </robot>

File: grizzly_ur10_description/urdf/grizzly_ur10.urdf (robot description, URDF)
Before this commit: robot grizzly_ur10, 61 links, 60 joints
Links:
- removed link grizzly_ur10_kinect_frame
- removed link grizzly_ur10_kinect_optical_frame
- link back_left_wheel: geometry collision cylinder length=0.2772 radius=0.33; visual mesh filename=package://grizzly_description/meshes/wheel.stl
- link back_right_wheel: geometry collision cylinder length=0.2772 radius=0.33; visual mesh filename=package://grizzly_description/meshes/wheel.stl
- link front_left_wheel: geometry collision cylinder length=0.2772 radius=0.33; visual mesh filename=package://grizzly_description/meshes/wheel.stl
- link front_right_wheel: geometry collision cylinder length=0.2772 radius=0.33; visual mesh filename=package://grizzly_description/meshes/wheel.stl
Joints:
- removed joint grizzly_ur10_kinect_frame_joint
- removed joint grizzly_ur10_kinect_optical_joint
